Commit message: Deleting some garbadge

File: src/omnibot_description/urdf/roller.xacro (robot description, xacro)
@@ -23,4 +23,5 @@
                     <mesh filename="package://omnibot_description/meshes/wheel/colision_omni_roller.stl"/>
                 </geometry>
+            </collision>
         </link>
         <joint name="roller_${wheel_id}_${id}_joint" type="continuous">
