Commit message: launch file for description added

File: src/omnibot_description/urdf/omnibot.urdf.xacro (robot description, xacro)
@@ -16,4 +16,6 @@
         <origin rpy="0 0 0" xyz="0 0 0.03"/>
     </joint>
-    <xacro:wheel number="1" pitch="45" x="0" y="0.0955" z="-0.0124"/>
+    <xacro:wheel number="1" yaw="0" x="0" y="0.0955"/>
+    <xacro:wheel number="2" yaw="2.085" x="-0.0828" y="-0.0475"/>
+    <xacro:wheel number="3" yaw="-2.085" x="0.0828" y="-0.048"/>
 </robot>

File: src/omnibot_description/urdf/roller.xacro (robot description, xacro)
@@ -5,5 +5,5 @@
     </material>
     <xacro:macro name="roller" params="number parent_number pitch x y z">
-        <link name="roller_${number}_link">
+        <link name="roller_${parent_number}_${number}_link">
             <visual>
                 <origin rpy="0 0 0" xyz="0 0 0"/>
@@ -14,7 +14,7 @@
             </visual>
         </link>
-        <joint name="roller_${number}_joint" type="continuous">
+        <joint name="roller_${parent_number}_${number}_joint" type="continuous">
             <parent link="wheel_${parent_number}_link"/>
-            <child link="roller_${number}_link"/>
+            <child link="roller_${parent_number}_${number}_link"/>
             <axis xyz="0 0 1"/>
             <origin rpy="0 ${pitch} 0" xyz="${x} ${y} ${z}"/>

File: src/omnibot_description/urdf/wheel.xacro (robot description, xacro)
@@ -5,5 +5,5 @@
         <color rgba="0.8 0.8 0.8 1.0"/>
     </material>
-    <xacro:macro name="wheel" params="number pitch x y z">
+    <xacro:macro name="wheel" params="number yaw x y">
         <link name="wheel_${number}_link">
             <visual>
@@ -19,5 +19,5 @@
             <child link="wheel_${number}_link"/>
             <axis xyz="0 1 0"/>
-            <origin rpy="0 ${pitch} 0" xyz="${x} ${y} ${z}"/>
+            <origin rpy="0 0 ${yaw}" xyz="${x} ${y} -0.0124"/>
         </joint>
         <xacro:roller number="1" parent_number="${number}" pitch="-0.257" x="-0.0285" y="-0.002" z="-0.0075"/>

Commit message: Colision missing inercia and such

File: src/omnibot_description/urdf/omnibot.urdf.xacro (robot description, xacro)
@@ -10,4 +10,10 @@
             </geometry>
         </visual>
+        <colision>
+            <origin rpy="0 0 0" xyz="0 0 0"/>
+            <geometry>
+                <mesh filename="package://omnibot_description/meshes/omni_bot_base.stl"/>
+            </geometry>
+        </colision>
     </link>
     <joint name="base_joint" type="fixed">

File: src/omnibot_description/urdf/roller.xacro (robot description, xacro)
@@ -13,4 +13,10 @@
                 <material name="green"/>
             </visual>
+            <colision>
+                <origin rpy="0 0 0" xyz="0 0 0"/>
+                <geometry>
+                    <mesh filename="package://omnibot_description/meshes/wheel/colision_omni_roller.stl"/>
+                </geometry>
+            </colision>
         </link>
         <joint name="roller_${parent_number}_${number}_joint" type="continuous">

File: src/omnibot_description/urdf/wheel.xacro (robot description, xacro)
@@ -8,5 +8,5 @@
         <link name="wheel_${number}_link">
             <visual>
-                <origin rpy="0 0 0" xyz="0 0 0"/>
+                <origin xyz="0 0 0" rpy="0 0 0"/>
                 <geometry>
                     <mesh filename="package://omnibot_description/meshes/wheel/wheel.stl"/>
@@ -14,4 +14,10 @@
                 <material name="gray"/>
             </visual>
+            <colision>
+                <origin rpy="1.58 0 0" xyz="0 0.005 0"/>
+                <geometry>
+                    <cylinder length="0.028" radius="0.036925"/>
+                </geometry>
+            </colision>
         </link>
         <joint name="wheel_${number}_joint" type="continuous">

Commit message: gazebo simulation not working

File: src/omnibot_description/urdf/omnibot.urdf.xacro (robot description, xacro)
@@ -1,7 +1,12 @@
 <?xml version="1.0"?>
 <robot xmlns:xacro="http://www.ros.org/wiki/xacro" name="omnibot">
-    <xacro:include filename="$(find omnibot_description)/urdf/wheel.xacro"/>
+    <xacro:include filename="$(find omnibot_description)/urdf/omnibot_gazebo.xacro"/>
     <link name="base_footprint"/>
     <link name="base_link">
+        <inertial>
+            <mass value="1.0"/>
+            <origin xyz="0 0 0" rpy="0 0 0"/>
+            <inertia ixx="0.001" ixy="0.0" ixz="0.0" iyy="0.001" iyz="0.0" izz="0.001"/>
+        </inertial>
         <visual>
             <origin rpy="0 0 0" xyz="0 0 0"/>
@@ -22,4 +27,5 @@
         <origin rpy="0 0 0" xyz="0 0 0.03"/>
     </joint>
+    <xacro:include filename="$(find omnibot_description)/urdf/wheel.xacro"/>
     <xacro:wheel number="1" yaw="0" x="0" y="0.0955"/>
     <xacro:wheel number="2" yaw="2.085" x="-0.0828" y="-0.0475"/>

File: src/omnibot_description/urdf/omnibot_gazebo.xacro (robot description, xacro)
@@ -1,3 +1,30 @@
 <?xml version="1.0"?>
-<robot xmlns:xacro="http://www.ros.org/wiki/xacro" name="omnibot">
+<robot name="omnibot" xmlns:xacro="http://www.ros.org/wiki/xacro">
+    <gazebo reference="wheel_1_link">
+        <mu1>100000000000000.0</mu1>
+        <mu2>100000000000000.0</mu2>
+        <kp>10000000000000.0</kp>
+        <kd>10.0</kd>
+        <minDepth>0.001</minDepth>
+        <maxVel>0.1</maxVel>
+        <fdir1>1 0 0</fdir1>
+    </gazebo>
+    <gazebo reference="wheel_2_link">
+        <mu1>1000000000000000.0</mu1><mu1>100000000000000.0</mu1>
+        <mu2>100000000000000.0</mu2>
+        <kp>10000000000000.0</kp>
+        <kd>10.0</kd>
+        <minDepth>0.001</minDepth>
+        <maxVel>0.1</maxVel>
+        <fdir1>1 0 0</fdir1>
+    </gazebo>
+    <gazebo reference="wheel_3_link">
+        <mu1>100000000000000.0</mu1>
+        <mu2>100000000000000.0</mu2>
+        <kp>10000000000000.0</kp>
+        <kd>10.0</kd>
+        <minDepth>0.001</minDepth>
+        <maxVel>0.1</maxVel>
+        <fdir1>1 0 0</fdir1>
+    </gazebo>
 </robot>

File: src/omnibot_description/urdf/roller.xacro (robot description, xacro)
@@ -6,4 +6,9 @@
     <xacro:macro name="roller" params="number parent_number pitch x y z">
         <link name="roller_${parent_number}_${number}_link">
+            <inertial>
+                <mass value="1.0"/>
+                <origin xyz="0 0 0" rpy="0 0 0"/>
+                <inertia ixx="0.001" ixy="0.0" ixz="0.0" iyy="0.001" iyz="0.0" izz="0.001"/>
+            </inertial>
             <visual>
                 <origin rpy="0 0 0" xyz="0 0 0"/>
@@ -16,5 +21,5 @@
                 <origin rpy="0 0 0" xyz="0 0 0"/>
                 <geometry>
-                    <mesh filename="package://omnibot_description/meshes/wheel/colision_omni_roller.stl"/>
+                    <sphere radius="0.0078"/>
                 </geometry>
             </colision>

File: src/omnibot_description/urdf/wheel.xacro (robot description, xacro)
@@ -7,4 +7,9 @@
     <xacro:macro name="wheel" params="number yaw x y">
         <link name="wheel_${number}_link">
+            <inertial>
+                <mass value="1.0"/>
+                <origin xyz="0 0 0" rpy="0 0 0"/>
+                <inertia ixx="0.001" ixy="0.0" ixz="0.0" iyy="0.001" iyz="0.0" izz="0.001"/>
+            </inertial>
             <visual>
                 <origin xyz="0 0 0" rpy="0 0 0"/>

Commit message: All good, interfacing with gazebo

File: src/omnibot_description/urdf/omnibot.urdf.xacro (robot description, xacro)
@@ -2,4 +2,5 @@
 <robot xmlns:xacro="http://www.ros.org/wiki/xacro" name="omnibot">
     <xacro:include filename="$(find omnibot_description)/urdf/omnibot_gazebo.xacro"/>
+    <xacro:include filename="$(find omnibot_description)/urdf/omnibot_ros2_control.xacro"/>
     <link name="base_footprint"/>
     <link name="base_link">
@@ -15,10 +16,10 @@
             </geometry>
         </visual>
-        <colision>
+        <collision>
             <origin rpy="0 0 0" xyz="0 0 0"/>
             <geometry>
                 <mesh filename="package://omnibot_description/meshes/omni_bot_base.stl"/>
             </geometry>
-        </colision>
+        </collision>
     </link>
     <joint name="base_joint" type="fixed">
@@ -28,6 +29,6 @@
     </joint>
     <xacro:include filename="$(find omnibot_description)/urdf/wheel.xacro"/>
-    <xacro:wheel number="1" yaw="0" x="0" y="0.0955"/>
-    <xacro:wheel number="2" yaw="2.085" x="-0.0828" y="-0.0475"/>
-    <xacro:wheel number="3" yaw="-2.085" x="0.0828" y="-0.048"/>
+    <xacro:wheel id="1" yaw="0" x="0" y="0.0955"/>
+    <xacro:wheel id="2" yaw="2.085" x="-0.0828" y="-0.0475"/>
+    <xacro:wheel id="3" yaw="-2.085" x="0.0828" y="-0.048"/>
 </robot>

File: src/omnibot_description/urdf/omnibot_gazebo.xacro (robot description, xacro)
@@ -1,30 +1,36 @@
 <?xml version="1.0"?>
 <robot name="omnibot" xmlns:xacro="http://www.ros.org/wiki/xacro">
-    <gazebo reference="wheel_1_link">
-        <mu1>100000000000000.0</mu1>
-        <mu2>100000000000000.0</mu2>
-        <kp>10000000000000.0</kp>
-        <kd>10.0</kd>
-        <minDepth>0.001</minDepth>
-        <maxVel>0.1</maxVel>
-        <fdir1>1 0 0</fdir1>
-    </gazebo>
-    <gazebo reference="wheel_2_link">
-        <mu1>1000000000000000.0</mu1><mu1>100000000000000.0</mu1>
-        <mu2>100000000000000.0</mu2>
-        <kp>10000000000000.0</kp>
-        <kd>10.0</kd>
-        <minDepth>0.001</minDepth>
-        <maxVel>0.1</maxVel>
-        <fdir1>1 0 0</fdir1>
-    </gazebo>
-    <gazebo reference="wheel_3_link">
-        <mu1>100000000000000.0</mu1>
-        <mu2>100000000000000.0</mu2>
-        <kp>10000000000000.0</kp>
-        <kd>10.0</kd>
-        <minDepth>0.001</minDepth>
-        <maxVel>0.1</maxVel>
-        <fdir1>1 0 0</fdir1>
+    <xacro:macro name="transmission" params="id">
+        <transmission name="wheel_${id}_transmission">
+            <plugin>transmission_interface/SimpleTransmission</plugin>
+            <actuator name="wheel_${id}_motor" role="actuator_${id}"/>
+            <joint name="wheel_${id}_joint" role="joint_${id}">
+                <mechanical_reduction>1.0</mechanical_reduction>
+            </joint>
+        </transmission>
+    </xacro:macro>
+    <xacro:transmission id="1"/>
+    <xacro:transmission id="2"/>
+    <xacro:transmission id="3"/>
+    <xacro:macro name="wheel_link_values" params="id">
+        <gazebo reference="wheel_${id}_link">
+            <mu1>100000000000000.0</mu1>
+            <mu2>100000000000000.0</mu2>
+            <kp>10000000000000.0</kp>
+            <kd>10.0</kd>
+            <minDepth>0.001</minDepth>
+            <maxVel>0.1</maxVel>
+            <fdir1>1 0 0</fdir1>
+        </gazebo>
+    </xacro:macro>
+    <xacro:wheel_link_values id="1"/>
+    <xacro:wheel_link_values id="2"/>
+    <xacro:wheel_link_values id="3"/>
+    <gazebo>
+        <plugin filename="libgazebo_ros2_control.so" name="gazebo_ros2_control">
+            <robot_param>robot_description</robot_param>
+            <robot_param_node>robot_state_publisher</robot_param_node>
+            <parameters>$(find omnibot_controller)/config/omnibot_controllers.yaml</parameters>
+        </plugin>
     </gazebo>
 </robot>

File: src/omnibot_description/urdf/roller.xacro (robot description, xacro)
@@ -4,6 +4,6 @@
         <color rgba="0 1 0 1.0"/>
     </material>
-    <xacro:macro name="roller" params="number parent_number pitch x y z">
-        <link name="roller_${parent_number}_${number}_link">
+    <xacro:macro name="roller" params="id parent_id pitch x y z">
+        <link name="roller_${parent_id}_${id}_link">
             <inertial>
                 <mass value="1.0"/>
@@ -18,14 +18,14 @@
                 <material name="green"/>
             </visual>
-            <colision>
+            <collision>
                 <origin rpy="0 0 0" xyz="0 0 0"/>
                 <geometry>
                     <sphere radius="0.0078"/>
                 </geometry>
-            </colision>
+            </collision>
         </link>
-        <joint name="roller_${parent_number}_${number}_joint" type="continuous">
-            <parent link="wheel_${parent_number}_link"/>
-            <child link="roller_${parent_number}_${number}_link"/>
+        <joint name="roller_${parent_id}_${id}_joint" type="continuous">
+            <parent link="wheel_${parent_id}_link"/>
+            <child link="roller_${parent_id}_${id}_link"/>
             <axis xyz="0 0 1"/>
             <origin rpy="0 ${pitch} 0" xyz="${x} ${y} ${z}"/>

File: src/omnibot_description/urdf/wheel.xacro (robot description, xacro)
@@ -5,6 +5,6 @@
         <color rgba="0.8 0.8 0.8 1.0"/>
     </material>
-    <xacro:macro name="wheel" params="number yaw x y">
-        <link name="wheel_${number}_link">
+    <xacro:macro name="wheel" params="id yaw x y">
+        <link name="wheel_${id}_link">
             <inertial>
                 <mass value="1.0"/>
@@ -19,29 +19,29 @@
                 <material name="gray"/>
             </visual>
-            <colision>
+            <collision>
                 <origin rpy="1.58 0 0" xyz="0 0.005 0"/>
                 <geometry>
                     <cylinder length="0.028" radius="0.036925"/>
                 </geometry>
-            </colision>
+            </collision>
         </link>
-        <joint name="wheel_${number}_joint" type="continuous">
+        <joint name="wheel_${id}_joint" type="continuous">
             <parent link="base_link"/>
-            <child link="wheel_${number}_link"/>
+            <child link="wheel_${id}_link"/>
             <axis xyz="0 1 0"/>
             <origin rpy="0 0 ${yaw}" xyz="${x} ${y} -0.0124"/>
         </joint>
-        <xacro:roller number="1" parent_number="${number}" pitch="-0.257" x="-0.0285" y="-0.002" z="-0.0075"/>
-        <xacro:roller number="2" parent_number="${number}" pitch="-1.3" x="-0.0079" y="-0.002" z="-0.0283"/>
-        <xacro:roller number="3" parent_number="${number}" pitch="0.789" x="0.0206" y="-0.002" z="-0.0208"/>
-        <xacro:roller number="4" parent_number="${number}" pitch="-0.257" x="0.0285" y="-0.002" z="0.0075"/>
-        <xacro:roller number="5" parent_number="${number}" pitch="-1.3" x="0.0079" y="-0.002" z="0.0283"/>
-        <xacro:roller number="6" parent_number="${number}" pitch="0.789" x="-0.0206" y="-0.002" z="0.0208"/>
-        <xacro:roller number="7" parent_number="${number}" pitch="0.25" x="-0.0286" y="0.0122" z="0.0075"/>
-        <xacro:roller number="8" parent_number="${number}" pitch="-0.8" x="-0.0205" y="0.0122" z="-0.021"/>
-        <xacro:roller number="9" parent_number="${number}" pitch="-1.85" x="0.008" y="0.0122" z="-0.0285"/>
-        <xacro:roller number="10" parent_number="${number}" pitch="0.25" x="0.0286" y="0.0122" z="-0.0075"/>
-        <xacro:roller number="11" parent_number="${number}" pitch="-0.8" x="0.0205" y="0.0122" z="0.021"/>
-        <xacro:roller number="12" parent_number="${number}" pitch="-1.85" x="-0.008" y="0.0122" z="0.0285"/>
+        <xacro:roller id="1" parent_id="${id}" pitch="-0.257" x="-0.0285" y="-0.002" z="-0.0075"/>
+        <xacro:roller id="2" parent_id="${id}" pitch="-1.3" x="-0.0079" y="-0.002" z="-0.0283"/>
+        <xacro:roller id="3" parent_id="${id}" pitch="0.789" x="0.0206" y="-0.002" z="-0.0208"/>
+        <xacro:roller id="4" parent_id="${id}" pitch="-0.257" x="0.0285" y="-0.002" z="0.0075"/>
+        <xacro:roller id="5" parent_id="${id}" pitch="-1.3" x="0.0079" y="-0.002" z="0.0283"/>
+        <xacro:roller id="6" parent_id="${id}" pitch="0.789" x="-0.0206" y="-0.002" z="0.0208"/>
+        <xacro:roller id="7" parent_id="${id}" pitch="0.25" x="-0.0286" y="0.0122" z="0.0075"/>
+        <xacro:roller id="8" parent_id="${id}" pitch="-0.8" x="-0.0205" y="0.0122" z="-0.021"/>
+        <xacro:roller id="9" parent_id="${id}" pitch="-1.85" x="0.008" y="0.0122" z="-0.0285"/>
+        <xacro:roller id="10" parent_id="${id}" pitch="0.25" x="0.0286" y="0.0122" z="-0.0075"/>
+        <xacro:roller id="11" parent_id="${id}" pitch="-0.8" x="0.0205" y="0.0122" z="0.021"/>
+        <xacro:roller id="12" parent_id="${id}" pitch="-1.85" x="-0.008" y="0.0122" z="0.0285"/>
     </xacro:macro>
 </robot>

Commit message: Trying new onshape solution for simulation

File: src/omnibot_description/urdf/omnibot.urdf.xacro (robot description, xacro)
@@ -5,13 +5,8 @@
     <link name="base_footprint"/>
     <link name="base_link">
-        <inertial>
-            <mass value="1.0"/>
-            <origin xyz="0 0 0" rpy="0 0 0"/>
-            <inertia ixx="0.001" ixy="0.0" ixz="0.0" iyy="0.001" iyz="0.0" izz="0.001"/>
-        </inertial>
         <visual>
             <origin rpy="0 0 0" xyz="0 0 0"/>
             <geometry>
-                <mesh filename="package://omnibot_description/meshes/omni_bot_base.stl"/>
+                <mesh filename="package://omnibot_description/meshes/base.stl"/>
             </geometry>
         </visual>
@@ -22,9 +17,14 @@
             </geometry>
         </collision>
+        <inertial>
+            <origin xyz="5.7125161491566575863e-17 -6.5024821714209305867e-17 0.0080527486487109532082" rpy="0 0 0"/>
+            <mass value="0.33121488483749478293" />
+            <inertia ixx="0.0012461406422939467261" ixy="0"  ixz="0" iyy="0.0012461406422939458587" iyz="0" izz="0.0024316574431770781976" />
+        </inertial>
     </link>
     <joint name="base_joint" type="fixed">
         <parent link="base_footprint"/>
         <child link="base_link"/>
-        <origin rpy="0 0 0" xyz="0 0 0.03"/>
+        <origin rpy="0 0 0" xyz="0 0 0.0"/>
     </joint>
     <xacro:include filename="$(find omnibot_description)/urdf/wheel.xacro"/>

File: src/omnibot_description/urdf/roller.xacro (robot description, xacro)
@@ -7,7 +7,7 @@
         <link name="roller_${parent_id}_${id}_link">
             <inertial>
-                <mass value="1.0"/>
-                <origin xyz="0 0 0" rpy="0 0 0"/>
-                <inertia ixx="0.001" ixy="0.0" ixz="0.0" iyy="0.001" iyz="0.0" izz="0.001"/>
+                <origin xyz="4.0756135840652012993e-11 8.4957117072138698775e-11 2.4283850775576134338e-11" rpy="0 0 0"/>
+                <mass value="0.0037899803393768708749" />
+                <inertia ixx="1.8303635244743848899e-07" ixy="4.2716081106694475295e-16"  ixz="-1.7514569765292920798e-15" iyy="1.830363607521377626e-07" iyz="-3.3429142897629588724e-15" izz="9.8097062080638907831e-08" />
             </inertial>
             <visual>
@@ -21,5 +21,5 @@
                 <origin rpy="0 0 0" xyz="0 0 0"/>
                 <geometry>
-                    <sphere radius="0.0078"/>
+                    <mesh filename="package://omnibot_description/meshes/wheel/colision_omni_roller.stl"/>
                 </geometry>
             </collision>

File: src/omnibot_description/urdf/wheel.xacro (robot description, xacro)
@@ -7,9 +7,4 @@
     <xacro:macro name="wheel" params="id yaw x y">
         <link name="wheel_${id}_link">
-            <inertial>
-                <mass value="1.0"/>
-                <origin xyz="0 0 0" rpy="0 0 0"/>
-                <inertia ixx="0.001" ixy="0.0" ixz="0.0" iyy="0.001" iyz="0.0" izz="0.001"/>
-            </inertial>
             <visual>
                 <origin xyz="0 0 0" rpy="0 0 0"/>
@@ -25,4 +20,9 @@
                 </geometry>
             </collision>
+            <inertial>
+                <origin xyz="-9.4588917160583760242e-06 -8.8415141495200006669e-06 -0.015131125342708530435" rpy="0 0 0"/>
+                <mass value="0.019223052335254620093" />
+                <inertia ixx="5.399262953463332839e-06" ixy="-7.3246329002135788826e-08"  ixz="-1.2642889979755781e-09" iyy="5.6557979176500377362e-06" iyz="1.9098649289524068763e-09" izz="8.6846392930505500327e-06" />
+            </inertial>
         </link>
         <joint name="wheel_${id}_joint" type="continuous">

Commit message: Trying new onshape solution for simulation

File: src/omnibot_description/urdf/omnibot.urdf.xacro (robot description, xacro)
@@ -6,7 +6,7 @@
     <link name="base_link">
         <inertial>
-            <mass value="1.0"/>
-            <origin xyz="0 0 0" rpy="0 0 0"/>
-            <inertia ixx="0.001" ixy="0.0" ixz="0.0" iyy="0.001" iyz="0.0" izz="0.001"/>
+            <origin xyz="0 0 0.04" rpy="0.0 0.25 0.3"/>
+            <mass value="8.2573504e-01"/>
+            <inertia ixx="2.2124416e-02" ixy="-1.2294101e-04" ixz="3.4938785e-04" iyy="2.1193702e-02" iyz="-5.0120904e-05" izz="2.0064271e-02"/>
         </inertial>
         <visual>

File: src/omnibot_description/urdf/roller.xacro (robot description, xacro)
@@ -21,5 +21,5 @@
                 <origin rpy="0 0 0" xyz="0 0 0"/>
                 <geometry>
-                    <sphere radius="0.0078"/>
+                    <mesh filename="package://omnibot_description/meshes/wheel/colision_omni_roller.stl"/>
                 </geometry>
             </collision>

File: src/omnibot_description/urdf/wheel.xacro (robot description, xacro)
@@ -7,9 +7,4 @@
     <xacro:macro name="wheel" params="id yaw x y">
         <link name="wheel_${id}_link">
-            <inertial>
-                <mass value="1.0"/>
-                <origin xyz="0 0 0" rpy="0 0 0"/>
-                <inertia ixx="0.001" ixy="0.0" ixz="0.0" iyy="0.001" iyz="0.0" izz="0.001"/>
-            </inertial>
             <visual>
                 <origin xyz="0 0 0" rpy="0 0 0"/>
