Commit message: Gazebo not working

File: src/omnibot_description/urdf/omnibot.urdf.xacro (robot description, xacro)
@@ -1,34 +1,1291 @@
 <?xml version="1.0"?>
 <robot xmlns:xacro="http://www.ros.org/wiki/xacro" name="omnibot">
-    <xacro:include filename="$(find omnibot_description)/urdf/omnibot_gazebo.xacro"/>
-    <xacro:include filename="$(find omnibot_description)/urdf/omnibot_ros2_control.xacro"/>
-    <link name="base_footprint"/>
-    <link name="base_link">
-        <visual>
-            <origin rpy="0 0 0" xyz="0 0 0"/>
-            <geometry>
-                <mesh filename="package://omnibot_description/meshes/base.stl"/>
-            </geometry>
-        </visual>
-        <collision>
-            <origin rpy="0 0 0" xyz="0 0 0"/>
-            <geometry>
-                <mesh filename="package://omnibot_description/meshes/omni_bot_base.stl"/>
-            </geometry>
-        </collision>
-        <inertial>
-            <origin xyz="5.7125161491566575863e-17 -6.5024821714209305867e-17 0.0080527486487109532082" rpy="0 0 0"/>
-            <mass value="0.33121488483749478293" />
-            <inertia ixx="0.0012461406422939467261" ixy="0"  ixz="0" iyy="0.0012461406422939458587" iyz="0" izz="0.0024316574431770781976" />
-        </inertial>
-    </link>
-    <joint name="base_joint" type="fixed">
-        <parent link="base_footprint"/>
-        <child link="base_link"/>
-        <origin rpy="0 0 0" xyz="0 0 0.0"/>
-    </joint>
-    <xacro:include filename="$(find omnibot_description)/urdf/wheel.xacro"/>
-    <xacro:wheel id="1" yaw="0" x="0" y="0.0955"/>
-    <xacro:wheel id="2" yaw="2.085" x="-0.0828" y="-0.0475"/>
-    <xacro:wheel id="3" yaw="-2.085" x="0.0828" y="-0.048"/>
+<link name="base_footprint"></link>
+<joint name="base_footprint_to_base" type="fixed">
+<parent link="base_footprint"/>
+<child link="base" />
+<origin rpy="0.0 0 0" xyz="0 0 0"/>
+</joint>
+<link name="base">
+<visual>
+<origin xyz="0 0 0" rpy="0 -0 0" />
+<geometry>
+<mesh filename="package://omnibot_description/meshes/base.stl"/>
+</geometry>
+<material name="base_material">
+<color rgba="0.98039215686274505668 0.71372549019607844922 0.0039215686274509803377 1.0"/>
+</material>
+</visual>
+<collision>
+<origin xyz="0 0 0" rpy="0 -0 0" />
+<geometry>
+<mesh filename="package://omnibot_description/meshes/base.stl"/>
+</geometry>
+</collision>
+<inertial>
+<origin xyz="5.39784201477161138e-17 -6.6623166523784156457e-17 0.0080527486487109514735" rpy="0 0 0"/>
+<mass value="0.33121488483749472742" />
+<inertia ixx="0.0012461406422939471598" ixy="0"  ixz="0" iyy="0.0012461406422939458587" iyz="0" izz="0.0024316574431770786313" />
+</inertial>
+</link>
+<link name="motor">
+<visual>
+<origin xyz="0 0 0" rpy="0 -0 0" />
+<geometry>
+<mesh filename="package://omnibot_description/meshes/motor.stl"/>
+</geometry>
+<material name="motor_material">
+<color rgba="0.90196078431372550543 0.91764705882352937127 0.92941176470588238168 1.0"/>
+</material>
+</visual>
+<collision>
+<origin xyz="0 0 0" rpy="0 -0 0" />
+<geometry>
+<mesh filename="package://omnibot_description/meshes/motor.stl"/>
+</geometry>
+</collision>
+<inertial>
+<origin xyz="-2.0988305528124570607e-06 0.015050377580170260991 -0.021659280060218950859" rpy="0 0 0"/>
+<mass value="0.12860494827495116965" />
+<inertia ixx="4.6506247208995554765e-05" ixy="1.6921131916578434541e-09"  ixz="-3.460842774139133976e-09" iyy="4.6246527094885937542e-05" iyz="1.0074294037198123246e-06" izz="1.0661244977443992313e-05" />
+</inertial>
+</link>
+<link name="wheel">
+<visual>
+<origin xyz="0 0 0" rpy="0 -0 0" />
+<geometry>
+<mesh filename="package://omnibot_description/meshes/wheel.stl"/>
+</geometry>
+<material name="wheel_material">
+<color rgba="0.93784246287025563316 0.77727352216680201114 0.24802940574315229805 1.0"/>
+</material>
+</visual>
+<collision>
+<origin xyz="0 0 0" rpy="0 -0 0" />
+<geometry>
+<mesh filename="package://omnibot_description/meshes/wheel.stl"/>
+</geometry>
+</collision>
+<inertial>
+<origin xyz="-9.4588917160587250018e-06 -8.8415141495200853702e-06 -0.01513112534270852523" rpy="0 0 0"/>
+<mass value="0.019223052335254627032" />
+<inertia ixx="5.399262953463331145e-06" ixy="-7.3246329002135682946e-08"  ixz="-1.2642889979755847175e-09" iyy="5.6557979176500394302e-06" iyz="1.9098649289524134937e-09" izz="8.6846392930505500327e-06" />
+</inertial>
+</link>
+<link name="roller">
+<visual>
+<origin xyz="0 0 0" rpy="0 -0 0" />
+<geometry>
+<mesh filename="package://omnibot_description/meshes/roller.stl"/>
+</geometry>
+<material name="roller_material">
+<color rgba="0.098039215686274508443 0.098039215686274508443 0.098039215686274508443 1.0"/>
+</material>
+</visual>
+<collision>
+<origin xyz="0 0 0" rpy="0 -0 0" />
+<geometry>
+<mesh filename="package://omnibot_description/meshes/roller.stl"/>
+</geometry>
+</collision>
+<inertial>
+<origin xyz="4.075613575648331605e-11 8.4957116973785579774e-11 2.4283850935942104983e-11" rpy="0 0 0"/>
+<mass value="0.0037899803393768713086" />
+<inertia ixx="1.8303635244743846252e-07" ixy="4.2716081055023346446e-16"  ixz="-1.7514569747251380017e-15" iyy="1.830363607521377626e-07" iyz="-3.342914289645813028e-15" izz="9.8097062080638894596e-08" />
+</inertial>
+</link>
+<joint name="roller2_1" type="continuous">
+<origin xyz="0.020681564833504317152 -0.021119421197575767579 -0.010000000285351307028" rpy="1.570796326794896336 -0.6597090063277464278 2.3457233385922444668" />
+<parent link="wheel" />
+<child link="roller" />
+<axis xyz="0 0 1"/>
+<limit effort="1" velocity="20" />
+<joint_properties friction="0.0"/>
+</joint>
+<link name="roller_2">
+<visual>
+<origin xyz="0 0 0" rpy="0 -0 0" />
+<geometry>
+<mesh filename="package://omnibot_description/meshes/roller.stl"/>
+</geometry>
+<material name="roller_2_material">
+<color rgba="0.098039215686274508443 0.098039215686274508443 0.098039215686274508443 1.0"/>
+</material>
+</visual>
+<collision>
+<origin xyz="0 0 0" rpy="0 -0 0" />
+<geometry>
+<mesh filename="package://omnibot_description/meshes/roller.stl"/>
+</geometry>
+</collision>
+<inertial>
+<origin xyz="4.0756121878695495311e-11 8.4957096157103868053e-11 2.4283853104346449954e-11" rpy="0 0 0"/>
+<mass value="0.0037899803393768713086" />
+<inertia ixx="1.8303635244743851546e-07" ixy="4.2716078406856701082e-16"  ixz="-1.7514569792380156029e-15" iyy="1.8303636075213770966e-07" iyz="-3.3429143017915419041e-15" izz="9.8097062080638921065e-08" />
+</inertial>
+</link>
+<joint name="roller2_2" type="continuous">
+<origin xyz="0.028630754033681701104 0.0073511498047736482941 -0.01000000048162325017" rpy="-1.57079632679489678 -0.95923833802399638415 -2.8902645323988411796" />
+<parent link="wheel" />
+<child link="roller_2" />
+<axis xyz="0 0 1"/>
+<limit effort="1" velocity="20" />
+<joint_properties friction="0.0"/>
+</joint>
+<link name="roller_3">
+<visual>
+<origin xyz="0 0 0" rpy="0 -0 0" />
+<geometry>
+<mesh filename="package://omnibot_description/meshes/roller.stl"/>
+</geometry>
+<material name="roller_3_material">
+<color rgba="0.098039215686274508443 0.098039215686274508443 0.098039215686274508443 1.0"/>
+</material>
+</visual>
+<collision>
+<origin xyz="0 0 0" rpy="0 -0 0" />
+<geometry>
+<mesh filename="package://omnibot_description/meshes/roller.stl"/>
+</geometry>
+</collision>
+<inertial>
+<origin xyz="4.0756135756483322513e-11 8.4957089218209964145e-11 2.4283849201218619313e-11" rpy="0 0 0"/>
+<mass value="0.0037899803393768713086" />
+<inertia ixx="1.8303635244743851546e-07" ixy="4.2716080575839270692e-16"  ixz="-1.7514569852018300788e-15" iyy="1.8303636075213781554e-07" iyz="-3.3429143192620515193e-15" izz="9.8097062080638921065e-08" />
+</inertial>
+</link>
+<joint name="roller2_3" type="continuous">
+<origin xyz="0.020599080645981818899 0.021035055769849139717 -0.024199995144404309877" rpy="1.570796326794896558 -1.0050751734414828942 0.79586976703605405437" />
+<parent link="wheel" />
+<child link="roller_3" />
+<axis xyz="0 0 1"/>
+<limit effort="1" velocity="20" />
+<joint_properties friction="0.0"/>
+</joint>
+<link name="roller_4">
+<visual>
+<origin xyz="0 0 0" rpy="0 -0 0" />
+<geometry>
+<mesh filename="package://omnibot_description/meshes/roller.stl"/>
+</geometry>
+<material name="roller_4_material">
+<color rgba="0.098039215686274508443 0.098039215686274508443 0.098039215686274508443 1.0"/>
+</material>
+</visual>
+<collision>
+<origin xyz="0 0 0" rpy="0 -0 0" />
+<geometry>
+<mesh filename="package://omnibot_description/meshes/roller.stl"/>
+</geometry>
+</collision>
+<inertial>
+<origin xyz="4.0756135756483322513e-11 8.4957103095997810734e-11 2.4283847466495146567e-11" rpy="0 0 0"/>
+<mass value="0.0037899803393768713086" />
+<inertia ixx="1.8303635244743851546e-07" ixy="4.271608087105491898e-16"  ixz="-1.7514569813020677949e-15" iyy="1.8303636075213792142e-07" iyz="-3.3429143108588176171e-15" izz="9.8097062080638894596e-08" />
+</inertial>
+</link>
+<joint name="roller2_4" type="continuous">
+<origin xyz="0.0079490519369571598085 0.028470515462351391606 -0.00999999706275848943" rpy="1.570796326794896558 1.0765431582887567963 -1.8430676189349801675" />
+<parent link="wheel" />
+<child link="roller_4" />
+<axis xyz="0 0 1"/>
+<limit effort="1" velocity="20" />
+<joint_properties friction="0.0"/>
+</joint>
+<link name="roller_5">
+<visual>
+<origin xyz="0 0 0" rpy="0 -0 0" />
+<geometry>
+<mesh filename="package://omnibot_description/meshes/roller.stl"/>
+</geometry>
+<material name="roller_5_material">
+<color rgba="0.098039215686274508443 0.098039215686274508443 0.098039215686274508443 1.0"/>
+</material>
+</visual>
+<collision>
+<origin xyz="0 0 0" rpy="0 -0 0" />
+<geometry>
+<mesh filename="package://omnibot_description/meshes/roller.stl"/>
+</geometry>
+</collision>
+<inertial>
+<origin xyz="4.0756108000907706884e-11 8.495710309599777196e-11 2.4283849201218625775e-11" rpy="0 0 0"/>
+<mass value="0.0037899803393768713086" />
+<inertia ixx="1.8303635244743851546e-07" ixy="4.2716080992358075167e-16"  ixz="-1.7514569791668546301e-15" iyy="1.830363607521377626e-07" iyz="-3.3429143051782475935e-15" izz="9.8097062080638921065e-08" />
+</inertial>
+</link>
+<joint name="roller2_5" type="continuous">
+<origin xyz="-0.0079173874319013633205 0.028356888222933061133 -0.024199999101464753082" rpy="1.57079632679489678 -1.0027977690887008855 1.8430678811938736583" />
+<parent link="wheel" />
+<child link="roller_5" />
+<axis xyz="0 0 1"/>
+<limit effort="1" velocity="20" />
+<joint_properties friction="0.0"/>
+</joint>
+<link name="roller_6">
+<visual>
+<origin xyz="0 0 0" rpy="0 -0 0" />
+<geometry>
+<mesh filename="package://omnibot_description/meshes/roller.stl"/>
+</geometry>
+<material name="roller_6_material">
+<color rgba="0.098039215686274508443 0.098039215686274508443 0.098039215686274508443 1.0"/>
+</material>
+</visual>
+<collision>
+<origin xyz="0 0 0" rpy="0 -0 0" />
+<geometry>
+<mesh filename="package://omnibot_description/meshes/roller.stl"/>
+</geometry>
+</collision>
+<inertial>
+<origin xyz="4.0756114939801604328e-11 8.4957116973785579774e-11 2.4283850935942092058e-11" rpy="0 0 0"/>
+<mass value="0.0037899803393768713086" />
+<inertia ixx="1.8303635244743846252e-07" ixy="4.2716080625111133332e-16"  ixz="-1.7514569747251380017e-15" iyy="1.830363607521377626e-07" iyz="-3.3429143216676169799e-15" izz="9.8097062080638894596e-08" />
+</inertial>
+</link>
+<joint name="roller2_6" type="continuous">
+<origin xyz="-0.020681651273558431664 0.021119338664790682225 -0.010000000622266080885" rpy="1.57079632679489678 0.6597090063277464278 -0.7958693149975488712" />
+<parent link="wheel" />
+<child link="roller_6" />
+<axis xyz="0 0 1"/>
+<limit effort="1" velocity="20" />
+<joint_properties friction="0.0"/>
+</joint>
+<link name="roller_7">
+<visual>
+<origin xyz="0 0 0" rpy="0 -0 0" />
+<geometry>
+<mesh filename="package://omnibot_description/meshes/roller.stl"/>
+</geometry>
+<material name="roller_7_material">
+<color rgba="0.098039215686274508443 0.098039215686274508443 0.098039215686274508443 1.0"/>
+</material>
+</visual>
+<collision>
+<origin xyz="0 0 0" rpy="0 -0 0" />
+<geometry>
+<mesh filename="package://omnibot_description/meshes/roller.stl"/>
+</geometry>
+</collision>
+<inertial>
+<origin xyz="4.0756121878695514698e-11 8.495710309599777196e-11 2.428384443072907007e-11" rpy="0 0 0"/>
+<mass value="0.0037899803393768713086" />
+<inertia ixx="1.8303635244743851546e-07" ixy="4.2716080412586764471e-16"  ixz="-1.7514569793512011684e-15" iyy="1.830363607521377626e-07" iyz="-3.3429142984360687956e-15" izz="9.8097062080638894596e-08" />
+</inertial>
+</link>
+<joint name="roller2_7" type="continuous">
+<origin xyz="-0.028516458158703433812 0.0073218567028481632009 -0.024199999573447886214" rpy="-1.570796326794896558 -0.029118128194412656179 -0.25132764401667873067" />
+<parent link="wheel" />
+<child link="roller_7" />
+<axis xyz="0 0 1"/>
+<limit effort="1" velocity="20" />
+<joint_properties friction="0.0"/>
+</joint>
+<link name="roller_8">
+<visual>
+<origin xyz="0 0 0" rpy="0 -0 0" />
+<geometry>
+<mesh filename="package://omnibot_description/meshes/roller.stl"/>
+</geometry>
+<material name="roller_8_material">
+<color rgba="0.098039215686274508443 0.098039215686274508443 0.098039215686274508443 1.0"/>
+</material>
+</visual>
+<collision>
+<origin xyz="0 0 0" rpy="0 -0 0" />
+<geometry>
+<mesh filename="package://omnibot_description/meshes/roller.stl"/>
+</geometry>
+</collision>
+<inertial>
+<origin xyz="4.0756108000907706884e-11 8.4957096157103880977e-11 2.428385614011252322e-11" rpy="0 0 0"/>
+<mass value="0.0037899803393768713086" />
+<inertia ixx="1.8303635244743851546e-07" ixy="4.2716080575839270692e-16"  ixz="-1.7514569852018300788e-15" iyy="1.8303636075213781554e-07" iyz="-3.3429143192620515193e-15" izz="9.8097062080638921065e-08" />
+</inertial>
+</link>
+<joint name="roller2_8" type="continuous">
+<origin xyz="-0.02059908211981235221 -0.021035064443088044572 -0.02419999841828643361" rpy="1.570796326794896558 -1.0050751734414828942 0.79586976703605405437" />
+<parent link="wheel" />
+<child link="roller_8" />
+<axis xyz="0 0 1"/>
+<limit effort="1" velocity="20" />
+<joint_properties friction="0.0"/>
+</joint>
+<link name="roller_9">
+<visual>
+<origin xyz="0 0 0" rpy="0 -0 0" />
+<geometry>
+<mesh filename="package://omnibot_description/meshes/roller.stl"/>
+</geometry>
+<material name="roller_9_material">
+<color rgba="0.098039215686274508443 0.098039215686274508443 0.098039215686274508443 1.0"/>
+</material>
+</visual>
+<collision>
+<origin xyz="0 0 0" rpy="0 -0 0" />
+<geometry>
+<mesh filename="package://omnibot_description/meshes/roller.stl"/>
+</geometry>
+</collision>
+<inertial>
+<origin xyz="4.0756135756483303125e-11 8.4957116973785579774e-11 2.4283848333856884555e-11" rpy="0 0 0"/>
+<mass value="0.0037899803393768713086" />
+<inertia ixx="1.8303635244743851546e-07" ixy="4.2716076856204682185e-16"  ixz="-1.7514569736083902166e-15" iyy="1.830363607521377626e-07" iyz="-3.3429143097631856663e-15" izz="9.8097062080638921065e-08" />
+</inertial>
+</link>
+<joint name="roller2_9" type="continuous">
+<origin xyz="-0.028516433936169462149 -0.0073217973661773502747 -0.010000001453652984651" rpy="-1.570796326794896558 -0.95923833802399638415 -2.8902645323988411796" />
+<parent link="wheel" />
+<child link="roller_9" />
+<axis xyz="0 0 1"/>
+<limit effort="1" velocity="20" />
+<joint_properties friction="0.0"/>
+</joint>
+<link name="roller_10">
+<visual>
+<origin xyz="0 0 0" rpy="0 -0 0" />
+<geometry>
+<mesh filename="package://omnibot_description/meshes/roller.stl"/>
+</geometry>
+<material name="roller_10_material">
+<color rgba="0.098039215686274508443 0.098039215686274508443 0.098039215686274508443 1.0"/>
+</material>
+</visual>
+<collision>
+<origin xyz="0 0 0" rpy="0 -0 0" />
+<geometry>
+<mesh filename="package://omnibot_description/meshes/roller.stl"/>
+</geometry>
+</collision>
+<inertial>
+<origin xyz="4.0756149634271130327e-11 8.4957096157103893902e-11 2.4283849201218622544e-11" rpy="0 0 0"/>
+<mass value="0.0037899803393768713086" />
+<inertia ixx="1.8303635244743851546e-07" ixy="4.271608087105491898e-16"  ixz="-1.7514569813020677949e-15" iyy="1.8303636075213792142e-07" iyz="-3.3429143108588176171e-15" izz="9.8097062080638894596e-08" />
+</inertial>
+</link>
+<joint name="roller2_10" type="continuous">
+<origin xyz="-0.0082858436691589446021 -0.028375035936988014795 -0.010000003715208150012" rpy="1.570796326794896558 1.0765431582887567963 -1.8430676189349801675" />
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