Commit message: Finally interfaced

File: src/omnibot_description/urdf/omnibot.urdf.xacro (robot description, xacro)
@@ -26,7 +26,7 @@
 </collision>
 <inertial>
-<origin xyz="5.39784201477161138e-17 -6.6623166523784156457e-17 0.0080527486487109514735" rpy="0 0 0"/>
+<origin xyz="5.6525782187976014595e-17 -6.6023787220193582864e-17 0.0080527486487109532082" rpy="0 0 0"/>
 <mass value="0.33121488483749472742" />
-<inertia ixx="0.0012461406422939471598" ixy="0"  ixz="0" iyy="0.0012461406422939458587" iyz="0" izz="0.0024316574431770786313" />
+<inertia ixx="0.0012461406422939467261" ixy="0"  ixz="0" iyy="0.0012461406422939454251" iyz="0" izz="0.002431657443177077764" />
 </inertial>
 </link>
@@ -48,7 +48,7 @@
 </collision>
 <inertial>
-<origin xyz="-2.0988305528124570607e-06 0.015050377580170260991 -0.021659280060218950859" rpy="0 0 0"/>
-<mass value="0.12860494827495116965" />
-<inertia ixx="4.6506247208995554765e-05" ixy="1.6921131916578434541e-09"  ixz="-3.460842774139133976e-09" iyy="4.6246527094885937542e-05" iyz="1.0074294037198123246e-06" izz="1.0661244977443992313e-05" />
+<origin xyz="-2.0988305528124536725e-06 0.015050377580170260991 -0.021659280060218950859" rpy="0 0 0"/>
+<mass value="0.12860494827495119741" />
+<inertia ixx="4.6506247208995534436e-05" ixy="1.6921131916578382842e-09"  ixz="-3.4608427741391314945e-09" iyy="4.6246527094885930766e-05" iyz="1.0074294037198133834e-06" izz="1.066124497744399909e-05" />
 </inertial>
 </link>
@@ -60,5 +60,5 @@
 </geometry>
 <material name="wheel_material">
-<color rgba="0.93784246287025563316 0.77727352216680201114 0.24802940574315229805 1.0"/>
+<color rgba="0.93784246287025563316 0.77727352216680201114 0.24802940574315235356 1.0"/>
 </material>
 </visual>
@@ -70,7 +70,7 @@
 </collision>
 <inertial>
-<origin xyz="-9.4588917160587250018e-06 -8.8415141495200853702e-06 -0.01513112534270852523" rpy="0 0 0"/>
-<mass value="0.019223052335254627032" />
-<inertia ixx="5.399262953463331145e-06" ixy="-7.3246329002135682946e-08"  ixz="-1.2642889979755847175e-09" iyy="5.6557979176500394302e-06" iyz="1.9098649289524134937e-09" izz="8.6846392930505500327e-06" />
+<origin xyz="-9.458891716058550513e-06 -8.8415141495199108814e-06 -0.0151311253427085287" rpy="0 0 0"/>
+<mass value="0.019223052335254623563" />
+<inertia ixx="5.399262953463331145e-06" ixy="-7.3246329002135682946e-08"  ixz="-1.2642889979754722209e-09" iyy="5.6557979176500377362e-06" iyz="1.9098649289524929031e-09" izz="8.6846392930505483386e-06" />
 </inertial>
 </link>
@@ -92,7 +92,7 @@
 </collision>
 <inertial>
-<origin xyz="4.075613575648331605e-11 8.4957116973785579774e-11 2.4283850935942104983e-11" rpy="0 0 0"/>
-<mass value="0.0037899803393768713086" />
-<inertia ixx="1.8303635244743846252e-07" ixy="4.2716081055023346446e-16"  ixz="-1.7514569747251380017e-15" iyy="1.830363607521377626e-07" iyz="-3.342914289645813028e-15" izz="9.8097062080638894596e-08" />
+<origin xyz="4.0756135754373242931e-11 8.4957117021027906659e-11 2.4283851137571838313e-11" rpy="0 0 0"/>
+<mass value="0.0037899803393768708749" />
+<inertia ixx="1.8303635244743846252e-07" ixy="4.2716081056736456509e-16"  ixz="-1.7514569688045876161e-15" iyy="1.8303636075213773613e-07" iyz="-3.3429142877220179384e-15" izz="9.8097062080638907831e-08" />
 </inertial>
 </link>
@@ -122,7 +122,7 @@
 </collision>
 <inertial>
-<origin xyz="4.0756121878695495311e-11 8.4957096157103868053e-11 2.4283853104346449954e-11" rpy="0 0 0"/>
-<mass value="0.0037899803393768713086" />
-<inertia ixx="1.8303635244743851546e-07" ixy="4.2716078406856701082e-16"  ixz="-1.7514569792380156029e-15" iyy="1.8303636075213770966e-07" iyz="-3.3429143017915419041e-15" izz="9.8097062080638921065e-08" />
+<origin xyz="4.0756121876585422192e-11 8.4957096204346194938e-11 2.4283853305976183284e-11" rpy="0 0 0"/>
+<mass value="0.0037899803393768708749" />
+<inertia ixx="1.8303635244743851546e-07" ixy="4.2716078408569811146e-16"  ixz="-1.7514569733174652173e-15" iyy="1.8303636075213768319e-07" iyz="-3.3429142998677468145e-15" izz="9.80970620806389343e-08" />
 </inertial>
 </link>
@@ -152,7 +152,7 @@
 </collision>
 <inertial>
-<origin xyz="4.0756135756483322513e-11 8.4957089218209964145e-11 2.4283849201218619313e-11" rpy="0 0 0"/>
-<mass value="0.0037899803393768713086" />
-<inertia ixx="1.8303635244743851546e-07" ixy="4.2716080575839270692e-16"  ixz="-1.7514569852018300788e-15" iyy="1.8303636075213781554e-07" iyz="-3.3429143192620515193e-15" izz="9.8097062080638921065e-08" />
+<origin xyz="4.0756135754373249393e-11 8.4957089265452303955e-11 2.4283849402848352643e-11" rpy="0 0 0"/>
+<mass value="0.0037899803393768708749" />
+<inertia ixx="1.8303635244743851546e-07" ixy="4.2716080577552380755e-16"  ixz="-1.7514569792812796932e-15" iyy="1.8303636075213778907e-07" iyz="-3.3429143173382564297e-15" izz="9.80970620806389343e-08" />
 </inertial>
 </link>
@@ -182,7 +182,7 @@
 </collision>
 <inertial>
-<origin xyz="4.0756135756483322513e-11 8.4957103095997810734e-11 2.4283847466495146567e-11" rpy="0 0 0"/>
-<mass value="0.0037899803393768713086" />
-<inertia ixx="1.8303635244743851546e-07" ixy="4.271608087105491898e-16"  ixz="-1.7514569813020677949e-15" iyy="1.8303636075213792142e-07" iyz="-3.3429143108588176171e-15" izz="9.8097062080638894596e-08" />
+<origin xyz="4.0756135754373249393e-11 8.4957103143240124694e-11 2.4283847668124879897e-11" rpy="0 0 0"/>
+<mass value="0.0037899803393768708749" />
+<inertia ixx="1.8303635244743851546e-07" ixy="4.2716080872768029044e-16"  ixz="-1.7514569753815174093e-15" iyy="1.8303636075213789495e-07" iyz="-3.3429143089350225275e-15" izz="9.8097062080638907831e-08" />
 </inertial>
 </link>
@@ -212,7 +212,7 @@
 </collision>
 <inertial>
-<origin xyz="4.0756108000907706884e-11 8.495710309599777196e-11 2.4283849201218625775e-11" rpy="0 0 0"/>
-<mass value="0.0037899803393768713086" />
-<inertia ixx="1.8303635244743851546e-07" ixy="4.2716080992358075167e-16"  ixz="-1.7514569791668546301e-15" iyy="1.830363607521377626e-07" iyz="-3.3429143051782475935e-15" izz="9.8097062080638921065e-08" />
+<origin xyz="4.0756107998797633764e-11 8.4957103143240098845e-11 2.4283849402848359105e-11" rpy="0 0 0"/>
+<mass value="0.0037899803393768708749" />
+<inertia ixx="1.8303635244743851546e-07" ixy="4.2716080994071185231e-16"  ixz="-1.7514569732463042444e-15" iyy="1.8303636075213773613e-07" iyz="-3.342914303254452504e-15" izz="9.80970620806389343e-08" />
 </inertial>
 </link>
@@ -242,7 +242,7 @@
 </collision>
 <inertial>
-<origin xyz="4.0756114939801604328e-11 8.4957116973785579774e-11 2.4283850935942092058e-11" rpy="0 0 0"/>
-<mass value="0.0037899803393768713086" />
-<inertia ixx="1.8303635244743846252e-07" ixy="4.2716080625111133332e-16"  ixz="-1.7514569747251380017e-15" iyy="1.830363607521377626e-07" iyz="-3.3429143216676169799e-15" izz="9.8097062080638894596e-08" />
+<origin xyz="4.0756114937691531209e-11 8.4957117021027906659e-11 2.4283851137571825389e-11" rpy="0 0 0"/>
+<mass value="0.0037899803393768708749" />
+<inertia ixx="1.8303635244743846252e-07" ixy="4.2716080626824243395e-16"  ixz="-1.7514569688045876161e-15" iyy="1.8303636075213773613e-07" iyz="-3.3429143197438218903e-15" izz="9.8097062080638907831e-08" />
 </inertial>
 </link>
@@ -272,7 +272,7 @@
 </collision>
 <inertial>
-<origin xyz="4.0756121878695514698e-11 8.495710309599777196e-11 2.428384443072907007e-11" rpy="0 0 0"/>
-<mass value="0.0037899803393768713086" />
-<inertia ixx="1.8303635244743851546e-07" ixy="4.2716080412586764471e-16"  ixz="-1.7514569793512011684e-15" iyy="1.830363607521377626e-07" iyz="-3.3429142984360687956e-15" izz="9.8097062080638894596e-08" />
+<origin xyz="4.0756121876585441579e-11 8.4957103143240098845e-11 2.42838446323588034e-11" rpy="0 0 0"/>
+<mass value="0.0037899803393768708749" />
+<inertia ixx="1.8303635244743851546e-07" ixy="4.2716080414299874534e-16"  ixz="-1.7514569734306507828e-15" iyy="1.8303636075213773613e-07" iyz="-3.3429142965122737061e-15" izz="9.8097062080638907831e-08" />
 </inertial>
 </link>
@@ -302,7 +302,7 @@
 </collision>
 <inertial>
-<origin xyz="4.0756108000907706884e-11 8.4957096157103880977e-11 2.428385614011252322e-11" rpy="0 0 0"/>
-<mass value="0.0037899803393768713086" />
-<inertia ixx="1.8303635244743851546e-07" ixy="4.2716080575839270692e-16"  ixz="-1.7514569852018300788e-15" iyy="1.8303636075213781554e-07" iyz="-3.3429143192620515193e-15" izz="9.8097062080638921065e-08" />
+<origin xyz="4.0756107998797633764e-11 8.4957096204346207862e-11 2.428385634174225655e-11" rpy="0 0 0"/>
+<mass value="0.0037899803393768708749" />
+<inertia ixx="1.8303635244743851546e-07" ixy="4.2716080577552380755e-16"  ixz="-1.7514569792812796932e-15" iyy="1.8303636075213778907e-07" iyz="-3.3429143173382564297e-15" izz="9.80970620806389343e-08" />
 </inertial>
 </link>
@@ -332,7 +332,7 @@
 </collision>
 <inertial>
-<origin xyz="4.0756135756483303125e-11 8.4957116973785579774e-11 2.4283848333856884555e-11" rpy="0 0 0"/>
-<mass value="0.0037899803393768713086" />
-<inertia ixx="1.8303635244743851546e-07" ixy="4.2716076856204682185e-16"  ixz="-1.7514569736083902166e-15" iyy="1.830363607521377626e-07" iyz="-3.3429143097631856663e-15" izz="9.8097062080638921065e-08" />
+<origin xyz="4.0756135754373230006e-11 8.4957117021027906659e-11 2.4283848535486617886e-11" rpy="0 0 0"/>
+<mass value="0.0037899803393768708749" />
+<inertia ixx="1.8303635244743851546e-07" ixy="4.2716076857917792248e-16"  ixz="-1.751456967687839831e-15" iyy="1.8303636075213773613e-07" iyz="-3.3429143078393905768e-15" izz="9.80970620806389343e-08" />
 </inertial>
 </link>
@@ -362,7 +362,7 @@
 </collision>
 <inertial>
-<origin xyz="4.0756149634271130327e-11 8.4957096157103893902e-11 2.4283849201218622544e-11" rpy="0 0 0"/>
-<mass value="0.0037899803393768713086" />
-<inertia ixx="1.8303635244743851546e-07" ixy="4.271608087105491898e-16"  ixz="-1.7514569813020677949e-15" iyy="1.8303636075213792142e-07" iyz="-3.3429143108588176171e-15" izz="9.8097062080638894596e-08" />
+<origin xyz="4.0756149632161057208e-11 8.4957096204346220787e-11 2.4283849402848355874e-11" rpy="0 0 0"/>
+<mass value="0.0037899803393768708749" />
+<inertia ixx="1.8303635244743851546e-07" ixy="4.2716080872768029044e-16"  ixz="-1.7514569753815174093e-15" iyy="1.8303636075213789495e-07" iyz="-3.3429143089350225275e-15" izz="9.8097062080638907831e-08" />
 </inertial>
 </link>
@@ -392,7 +392,7 @@
 </collision>
 <inertial>
-<origin xyz="4.0756135756483322513e-11 8.4957110034891675867e-11 2.4283852670665571266e-11" rpy="0 0 0"/>
-<mass value="0.0037899803393768713086" />
-<inertia ixx="1.8303635244743851546e-07" ixy="4.2716080509708957469e-16"  ixz="-1.7514569804256685727e-15" iyy="1.830363607521377626e-07" iyz="-3.3429143165187155406e-15" izz="9.8097062080638921065e-08" />
+<origin xyz="4.0756135754373249393e-11 8.4957110082134002752e-11 2.4283852872295304596e-11" rpy="0 0 0"/>
+<mass value="0.0037899803393768708749" />
+<inertia ixx="1.8303635244743851546e-07" ixy="4.2716080511422067532e-16"  ixz="-1.7514569745051181871e-15" iyy="1.8303636075213773613e-07" iyz="-3.342914314594920451e-15" izz="9.80970620806389343e-08" />
 </inertial>
 </link>
@@ -422,7 +422,7 @@
 </collision>
 <inertial>
-<origin xyz="4.0756128817589418605e-11 8.4957103095997784884e-11 2.4283853538027309255e-11" rpy="0 0 0"/>
-<mass value="0.0037899803393768713086" />
-<inertia ixx="1.8303635244743851546e-07" ixy="4.2716081764220620394e-16"  ixz="-1.7514569798788242768e-15" iyy="1.8303636075213781554e-07" iyz="-3.3429143247134677051e-15" izz="9.8097062080638921065e-08" />
+<origin xyz="4.0756128815479345486e-11 8.495710314324011177e-11 2.4283853739657042585e-11" rpy="0 0 0"/>
+<mass value="0.0037899803393768708749" />
+<inertia ixx="1.8303635244743851546e-07" ixy="4.2716081765933730457e-16"  ixz="-1.7514569739582738912e-15" iyy="1.8303636075213778907e-07" iyz="-3.3429143227896726155e-15" izz="9.80970620806389343e-08" />
 </inertial>
 </link>
@@ -468,7 +468,7 @@
 </collision>
 <inertial>
-<origin xyz="-2.098830552821693955e-06 0.015050377580170260991 -0.021659280060218957797" rpy="0 0 0"/>
-<mass value="0.12860494827495116965" />
-<inertia ixx="4.6506247208995541212e-05" ixy="1.6921131916578171911e-09"  ixz="-3.4608427741392150397e-09" iyy="4.6246527094885937542e-05" iyz="1.0074294037198123246e-06" izz="1.0661244977443992313e-05" />
+<origin xyz="-2.0988305528216905668e-06 0.015050377580170260991 -0.021659280060218957797" rpy="0 0 0"/>
+<mass value="0.12860494827495119741" />
+<inertia ixx="4.6506247208995520883e-05" ixy="1.6921131916578120212e-09"  ixz="-3.4608427741392125582e-09" iyy="4.6246527094885930766e-05" iyz="1.0074294037198133834e-06" izz="1.066124497744399909e-05" />
 </inertial>
 </link>
@@ -480,5 +480,5 @@
 </geometry>
 <material name="wheel_2_material">
-<color rgba="0.93784246287025563316 0.77727352216680201114 0.24802940574315229805 1.0"/>
+<color rgba="0.93784246287025563316 0.77727352216680201114 0.24802940574315235356 1.0"/>
 </material>
 </visual>
@@ -490,7 +490,7 @@
 </collision>
 <inertial>
-<origin xyz="-9.4588917159859326844e-06 -8.8415141497943800495e-06 -0.015131125342709177486" rpy="0 0 0"/>
-<mass value="0.019223052335254627032" />
-<inertia ixx="5.3992629534639359265e-06" ixy="-7.3246329002134412397e-08"  ixz="-1.2642889980048933809e-09" iyy="5.655797917650548497e-06" iyz="1.9098649291001810383e-09" izz="8.6846392930512293531e-06" />
+<origin xyz="-9.4588917159859343785e-06 -8.841514149794161515e-06 -0.015131125342709179221" rpy="0 0 0"/>
+<mass value="0.019223052335254623563" />
+<inertia ixx="5.3992629534639359265e-06" ixy="-7.3246329002134650625e-08"  ixz="-1.2642889980048470588e-09" iyy="5.655797917650546803e-06" iyz="1.9098649291002472128e-09" izz="8.6846392930512276591e-06" />
 </inertial>
 </link>
@@ -512,7 +512,7 @@
 </collision>
 <inertial>
-<origin xyz="4.0756121878695508236e-11 8.495710309599777196e-11 2.4283850935942111445e-11" rpy="0 0 0"/>
-<mass value="0.0037899803393768713086" />
-<inertia ixx="1.8303635244743846252e-07" ixy="4.2716080818454802877e-16"  ixz="-1.7514569818893761193e-15" iyy="1.830363607521377626e-07" iyz="-3.3429143046647299098e-15" izz="9.8097062080638974005e-08" />
+<origin xyz="4.0756121876585435117e-11 8.4957103143240098845e-11 2.4283851137571844776e-11" rpy="0 0 0"/>
+<mass value="0.0037899803393768708749" />
+<inertia ixx="1.8303635244743846252e-07" ixy="4.2716080820167912941e-16"  ixz="-1.7514569759688257337e-15" iyy="1.8303636075213773613e-07" iyz="-3.3429143027409348202e-15" izz="9.809706208063898724e-08" />
 </inertial>
 </link>
@@ -542,7 +542,7 @@
 </collision>
 <inertial>
-<origin xyz="4.0756121878695514698e-11 8.4957089218209964145e-11 2.4283847466495149798e-11" rpy="0 0 0"/>
-<mass value="0.0037899803393768713086" />
-<inertia ixx="1.8303635244743851546e-07" ixy="4.2716081110329270245e-16"  ixz="-1.751456974632898271e-15" iyy="1.8303636075213770966e-07" iyz="-3.3429143064012541536e-15" izz="9.8097062080638921065e-08" />
+<origin xyz="4.0756121876585441579e-11 8.495708926545229103e-11 2.4283847668124883128e-11" rpy="0 0 0"/>
+<mass value="0.0037899803393768708749" />
+<inertia ixx="1.8303635244743851546e-07" ixy="4.2716081112042380309e-16"  ixz="-1.7514569687123478854e-15" iyy="1.8303636075213768319e-07" iyz="-3.3429143044774590641e-15" izz="9.80970620806389343e-08" />
 </inertial>
 </link>
@@ -572,7 +572,7 @@
 </collision>
 <inertial>
-<origin xyz="4.0756108000907706884e-11 8.495710309599777196e-11 2.4283849201218625775e-11" rpy="0 0 0"/>
-<mass value="0.0037899803393768713086" />
-<inertia ixx="1.8303635244743846252e-07" ixy="4.2716082629865883609e-16"  ixz="-1.751456982055647685e-15" iyy="1.830363607521377626e-07" iyz="-3.3429143072385219306e-15" izz="9.8097062080638921065e-08" />
+<origin xyz="4.0756107998797633764e-11 8.4957103143240098845e-11 2.4283849402848359105e-11" rpy="0 0 0"/>
+<mass value="0.0037899803393768708749" />
+<inertia ixx="1.8303635244743846252e-07" ixy="4.2716082631578993673e-16"  ixz="-1.7514569761350972994e-15" iyy="1.8303636075213773613e-07" iyz="-3.342914305314726841e-15" izz="9.80970620806389343e-08" />
 </inertial>
 </link>
@@ -602,7 +602,7 @@
 </collision>
 <inertial>
-<origin xyz="4.0756121878695514698e-11 8.4957089218209964145e-11 2.4283849201218625775e-11" rpy="0 0 0"/>
-<mass value="0.0037899803393768713086" />
-<inertia ixx="1.8303635244743851546e-07" ixy="4.2716081110329270245e-16"  ixz="-1.751456974632898271e-15" iyy="1.8303636075213770966e-07" iyz="-3.3429143064012541536e-15" izz="9.8097062080638921065e-08" />
+<origin xyz="4.0756121876585441579e-11 8.495708926545229103e-11 2.4283849402848359105e-11" rpy="0 0 0"/>
+<mass value="0.0037899803393768708749" />
+<inertia ixx="1.8303635244743851546e-07" ixy="4.2716081112042380309e-16"  ixz="-1.7514569687123478854e-15" iyy="1.8303636075213768319e-07" iyz="-3.3429143044774590641e-15" izz="9.80970620806389343e-08" />
 </inertial>
 </link>
@@ -632,7 +632,7 @@
 </collision>
 <inertial>
-<origin xyz="4.0756114939801610791e-11 8.4957103095997810734e-11 2.4283848333856891018e-11" rpy="0 0 0"/>
-<mass value="0.0037899803393768713086" />
-<inertia ixx="1.8303635244743851546e-07" ixy="4.2716081002607518111e-16"  ixz="-1.7514569688720561283e-15" iyy="1.8303636075213792142e-07" iyz="-3.3429143063932377491e-15" izz="9.8097062080638921065e-08" />
+<origin xyz="4.0756114937691537672e-11 8.4957103143240124694e-11 2.4283848535486624348e-11" rpy="0 0 0"/>
+<mass value="0.0037899803393768708749" />
+<inertia ixx="1.8303635244743851546e-07" ixy="4.2716081004320628175e-16"  ixz="-1.7514569629515057427e-15" iyy="1.8303636075213789495e-07" iyz="-3.3429143044694426595e-15" izz="9.80970620806389343e-08" />
 </inertial>
 </link>
@@ -662,7 +662,7 @@
 </collision>
 <inertial>
-<origin xyz="4.0756123613418984213e-11 8.4957089218209964145e-11 2.4283849201218625775e-11" rpy="0 0 0"/>
-<mass value="0.0037899803393768713086" />
-<inertia ixx="1.8303635244743851546e-07" ixy="4.2716080056066334142e-16"  ixz="-1.7514569719767807261e-15" iyy="1.8303636075213781554e-07" iyz="-3.3429143091577889585e-15" izz="9.8097062080638921065e-08" />
+<origin xyz="4.0756123611308911093e-11 8.4957089265452303955e-11 2.4283849402848359105e-11" rpy="0 0 0"/>
+<mass value="0.0037899803393768708749" />
+<inertia ixx="1.8303635244743851546e-07" ixy="4.2716080057779444205e-16"  ixz="-1.7514569660562303405e-15" iyy="1.8303636075213778907e-07" iyz="-3.342914307233993869e-15" izz="9.80970620806389343e-08" />
 </inertial>
 </link>
@@ -692,7 +692,7 @@
 </collision>
 <inertial>
-<origin xyz="4.0756108000907713346e-11 8.4957116973785592699e-11 2.4283847466495149798e-11" rpy="0 0 0"/>
-<mass value="0.0037899803393768713086" />
-<inertia ixx="1.8303635244743862134e-07" ixy="4.2716078752493109033e-16"  ixz="-1.751456982741181025e-15" iyy="1.8303636075213781554e-07" iyz="-3.3429143070805292629e-15" izz="9.8097062080638921065e-08" />
+<origin xyz="4.0756107998797640227e-11 8.4957117021027919584e-11 2.4283847668124883128e-11" rpy="0 0 0"/>
+<mass value="0.0037899803393768708749" />
+<inertia ixx="1.8303635244743862134e-07" ixy="4.2716078754206219097e-16"  ixz="-1.7514569768206306394e-15" iyy="1.8303636075213778907e-07" iyz="-3.3429143051567341733e-15" izz="9.80970620806389343e-08" />
 </inertial>
 </link>
@@ -722,7 +722,7 @@
 </collision>
 <inertial>
-<origin xyz="4.0756132287036357634e-11 8.4957089218209964145e-11 2.4283849201218625775e-11" rpy="0 0 0"/>
-<mass value="0.0037899803393768713086" />
-<inertia ixx="1.8303635244743846252e-07" ixy="4.2716079243101325436e-16"  ixz="-1.7514569849247919897e-15" iyy="1.8303636075213781554e-07" iyz="-3.3429143037005265246e-15" izz="9.8097062080638921065e-08" />
+<origin xyz="4.0756132284926284515e-11 8.4957089265452303955e-11 2.4283849402848359105e-11" rpy="0 0 0"/>
+<mass value="0.0037899803393768708749" />
+<inertia ixx="1.8303635244743846252e-07" ixy="4.27160792448144355e-16"  ixz="-1.7514569790042416041e-15" iyy="1.8303636075213778907e-07" iyz="-3.342914301776731435e-15" izz="9.80970620806389343e-08" />
 </inertial>
 </link>
@@ -752,7 +752,7 @@
 </collision>
 <inertial>
-<origin xyz="4.0756128817589418605e-11 8.4957103095997784884e-11 2.4283847466495149798e-11" rpy="0 0 0"/>
-<mass value="0.0037899803393768713086" />
-<inertia ixx="1.8303635244743846252e-07" ixy="4.2716080854255785807e-16"  ixz="-1.7514569700025312764e-15" iyy="1.8303636075213781554e-07" iyz="-3.3429143090399619327e-15" izz="9.8097062080638894596e-08" />
+<origin xyz="4.0756128815479345486e-11 8.495710314324011177e-11 2.4283847668124883128e-11" rpy="0 0 0"/>
+<mass value="0.0037899803393768708749" />
+<inertia ixx="1.8303635244743846252e-07" ixy="4.2716080855968895871e-16"  ixz="-1.7514569640819808907e-15" iyy="1.8303636075213778907e-07" iyz="-3.3429143071161668432e-15" izz="9.8097062080638907831e-08" />
 </inertial>
 </link>
@@ -782,7 +782,7 @@
 </collision>
 <inertial>
-<origin xyz="4.0756125348142460189e-11 8.4957103095997810734e-11 2.4283848333856887787e-11" rpy="0 0 0"/>
-<mass value="0.0037899803393768713086" />
-<inertia ixx="1.8303635244743846252e-07" ixy="4.2716080524040302003e-16"  ixz="-1.75145697758512797e-15" iyy="1.8303636075213792142e-07" iyz="-3.3429143052129578678e-15" izz="9.8097062080638921065e-08" />
+<origin xyz="4.075612534603238707e-11 8.4957103143240124694e-11 2.4283848535486621117e-11" rpy="0 0 0"/>
+<mass value="0.0037899803393768708749" />
+<inertia ixx="1.8303635244743846252e-07" ixy="4.2716080525753412066e-16"  ixz="-1.7514569716645775844e-15" iyy="1.8303636075213789495e-07" iyz="-3.3429143032891627782e-15" izz="9.80970620806389343e-08" />
 </inertial>
 </link>
@@ -812,7 +812,7 @@
 </collision>
 <inertial>
-<origin xyz="4.0756118409248569207e-11 8.4957116973785592699e-11 2.4283850935942098521e-11" rpy="0 0 0"/>
-<mass value="0.0037899803393768713086" />
-<inertia ixx="1.8303635244743851546e-07" ixy="4.2716081240888826617e-16"  ixz="-1.7514569720572778678e-15" iyy="1.8303636075213781554e-07" iyz="-3.3429143049916993444e-15" izz="9.8097062080638894596e-08" />
+<origin xyz="4.0756118407138496088e-11 8.4957117021027919584e-11 2.4283851137571831851e-11" rpy="0 0 0"/>
+<mass value="0.0037899803393768708749" />
+<inertia ixx="1.8303635244743851546e-07" ixy="4.271608124260193668e-16"  ixz="-1.7514569661367274822e-15" iyy="1.8303636075213778907e-07" iyz="-3.3429143030679042548e-15" izz="9.8097062080638907831e-08" />
 </inertial>
 </link>
@@ -842,7 +842,7 @@
 </collision>
 <inertial>
-<origin xyz="4.0756122312376383692e-11 8.4957089218209964145e-11 2.4283847466495149798e-11" rpy="0 0 0"/>
-<mass value="0.0037899803393768713086" />
-<inertia ixx="1.8303635244743851546e-07" ixy="4.2716080036563769716e-16"  ixz="-1.7514569771219131852e-15" iyy="1.830363607521377626e-07" iyz="-3.3429143156503039296e-15" izz="9.8097062080638894596e-08" />
+<origin xyz="4.0756122310266310573e-11 8.495708926545229103e-11 2.4283847668124883128e-11" rpy="0 0 0"/>
+<mass value="0.0037899803393768708749" />
+<inertia ixx="1.8303635244743851546e-07" ixy="4.2716080038276879779e-16"  ixz="-1.7514569712013627996e-15" iyy="1.8303636075213773613e-07" iyz="-3.34291431372650884e-15" izz="9.8097062080638907831e-08" />
 </inertial>
 </link>
@@ -888,7 +888,7 @@
 </collision>
 <inertial>
-<origin xyz="-2.0988305528127721569e-06 0.015050377580170262726 -0.021659280060218930042" rpy="0 0 0"/>
-<mass value="0.12860494827495116965" />
-<inertia ixx="4.6506247208995554765e-05" ixy="1.6921131916578407657e-09"  ixz="-3.4608427741353980148e-09" iyy="4.6246527094885937542e-05" iyz="1.0074294037198123246e-06" izz="1.0661244977443992313e-05" />
+<origin xyz="-2.0988305528127687688e-06 0.015050377580170262726 -0.021659280060218930042" rpy="0 0 0"/>
+<mass value="0.12860494827495119741" />
+<inertia ixx="4.6506247208995534436e-05" ixy="1.6921131916578355959e-09"  ixz="-3.4608427741353955333e-09" iyy="4.6246527094885930766e-05" iyz="1.0074294037198133834e-06" izz="1.066124497744399909e-05" />
 </inertial>
 </link>
@@ -900,5 +900,5 @@
 </geometry>
 <material name="wheel_3_material">
-<color rgba="0.93784246287025563316 0.77727352216680201114 0.24802940574315229805 1.0"/>
+<color rgba="0.93784246287025563316 0.77727352216680201114 0.24802940574315235356 1.0"/>
 </material>
 </visual>
@@ -910,7 +910,7 @@
 </collision>
 <inertial>
-<origin xyz="-9.4588917160631753129e-06 -8.8415141495136970477e-06 -0.015131125342708447168" rpy="0 0 0"/>
-<mass value="0.019223052335254627032" />
-<inertia ixx="5.3992629534633099691e-06" ixy="-7.3246329002137747589e-08"  ixz="-1.2642889979757766234e-09" iyy="5.6557979176500140192e-06" iyz="1.9098649289547163645e-09" izz="8.6846392930505551149e-06" />
+<origin xyz="-9.4588917160630008241e-06 -8.8415141495134344675e-06 -0.015131125342708447168" rpy="0 0 0"/>
+<mass value="0.019223052335254623563" />
+<inertia ixx="5.3992629534633099691e-06" ixy="-7.3246329002137853468e-08"  ixz="-1.2642889979757236838e-09" iyy="5.6557979176500131722e-06" iyz="1.9098649289547957739e-09" izz="8.6846392930505534208e-06" />
 </inertial>
 </link>
@@ -932,7 +932,7 @@
 </collision>
 <inertial>
-<origin xyz="4.0756121878695508236e-11 8.495710309599777196e-11 2.4283847466495140105e-11" rpy="0 0 0"/>
-<mass value="0.0037899803393768713086" />
-<inertia ixx="1.8303635244743851546e-07" ixy="4.2716079305631336652e-16"  ixz="-1.7514569699204268306e-15" iyy="1.8303636075213770966e-07" iyz="-3.3429143218139861765e-15" izz="9.8097062080638894596e-08" />
+<origin xyz="4.0756121876585435117e-11 8.4957103143240098845e-11 2.4283847668124873435e-11" rpy="0 0 0"/>
+<mass value="0.0037899803393768708749" />
+<inertia ixx="1.8303635244743851546e-07" ixy="4.2716079307344446715e-16"  ixz="-1.7514569639998764449e-15" iyy="1.8303636075213768319e-07" iyz="-3.342914319890191087e-15" izz="9.8097062080638907831e-08" />
 </inertial>
 </link>
@@ -962,7 +962,7 @@
 </collision>
 <inertial>
-<origin xyz="4.0756114939801610791e-11 8.4957075340422169256e-11 2.4283849201218625775e-11" rpy="0 0 0"/>
-<mass value="0.0037899803393768713086" />
-<inertia ixx="1.8303635244743851546e-07" ixy="4.2716079916151306517e-16"  ixz="-1.7514569851335445039e-15" iyy="1.8303636075213781554e-07" iyz="-3.3429143091482153426e-15" izz="9.8097062080638921065e-08" />
+<origin xyz="4.0756114937691537672e-11 8.4957075387664496141e-11 2.4283849402848359105e-11" rpy="0 0 0"/>
+<mass value="0.0037899803393768708749" />
+<inertia ixx="1.8303635244743851546e-07" ixy="4.271607991786441658e-16"  ixz="-1.7514569792129941183e-15" iyy="1.8303636075213778907e-07" iyz="-3.342914307224420253e-15" izz="9.80970620806389343e-08" />
 </inertial>
 </link>
@@ -992,7 +992,7 @@
 </collision>
 <inertial>
-<origin xyz="4.0756149634271130327e-11 8.4957103095997784884e-11 2.4283850935942104983e-11" rpy="0 0 0"/>
-<mass value="0.0037899803393768713086" />
-<inertia ixx="1.8303635244743851546e-07" ixy="4.2716081164325453214e-16"  ixz="-1.7514569778562385583e-15" iyy="1.8303636075213781554e-07" iyz="-3.3429142858942086828e-15" izz="9.8097062080638894596e-08" />
+<origin xyz="4.0756149632161057208e-11 8.495710314324011177e-11 2.4283851137571838313e-11" rpy="0 0 0"/>
+<mass value="0.0037899803393768708749" />
+<inertia ixx="1.8303635244743851546e-07" ixy="4.2716081166038563277e-16"  ixz="-1.7514569719356881727e-15" iyy="1.8303636075213778907e-07" iyz="-3.3429142839704135932e-15" izz="9.8097062080638907831e-08" />
 </inertial>
 </link>
@@ -1022,7 +1022,7 @@
 </collision>
 <inertial>
-<origin xyz="4.0756135756483322513e-11 8.4957103095997784884e-11 2.4283845731771677052e-11" rpy="0 0 0"/>
-<mass value="0.0037899803393768713086" />
-<inertia ixx="1.8303635244743851546e-07" ixy="4.2716081164325453214e-16"  ixz="-1.7514569778562385583e-15" iyy="1.8303636075213781554e-07" iyz="-3.3429142858942086828e-15" izz="9.8097062080638894596e-08" />
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