Commit message: Taking care of the create xacro script

File: src/omnibot_description/urdf/omnibot.urdf.xacro (robot description, xacro)
@@ -6,29 +6,7 @@
 <joint name="base_footprint_to_base" type="fixed">
 <parent link="base_footprint"/>
-<child link="base" />
+<child link="motor" />
 <origin rpy="0.0 0 0" xyz="0 0 0"/>
 </joint>
-<link name="base">
-<visual>
-<origin xyz="0 0 0" rpy="0 -0 0" />
-<geometry>
-<mesh filename="package://omnibot_description/meshes/base.stl"/>
-</geometry>
-<material name="base_material">
-<color rgba="0.98039215686274505668 0.71372549019607844922 0.0039215686274509803377 1.0"/>
-</material>
-</visual>
-<collision>
-<origin xyz="0 0 0" rpy="0 -0 0" />
-<geometry>
-<mesh filename="package://omnibot_description/meshes/base.stl"/>
-</geometry>
-</collision>
-<inertial>
-<origin xyz="5.6525782187976014595e-17 -6.6023787220193582864e-17 0.0080527486487109532082" rpy="0 0 0"/>
-<mass value="0.33121488483749472742" />
-<inertia ixx="0.0012461406422939467261" ixy="0"  ixz="0" iyy="0.0012461406422939454251" iyz="0" izz="0.002431657443177077764" />
-</inertial>
-</link>
 <link name="motor">
 <visual>
@@ -48,7 +26,7 @@
 </collision>
 <inertial>
-<origin xyz="-2.0988305528124536725e-06 0.015050377580170260991 -0.021659280060218950859" rpy="0 0 0"/>
-<mass value="0.12860494827495119741" />
-<inertia ixx="4.6506247208995534436e-05" ixy="1.6921131916578382842e-09"  ixz="-3.4608427741391314945e-09" iyy="4.6246527094885930766e-05" iyz="1.0074294037198133834e-06" izz="1.066124497744399909e-05" />
+<origin xyz="-0.083332409879302099531 -0.048114905775283510481 0.01775333870778863371" rpy="0 0 0"/>
+<mass value="0.11724467889003906129" />
+<inertia ixx="1.7177316862696019069e-05" ixy="-1.3512284026326213212e-05"  ixz="2.9006028519083257192e-07" iyy="3.2785367539480673885e-05" iyz="1.65594967207300257e-07" izz="4.052562608525466729e-05" />
 </inertial>
 </link>
@@ -60,5 +38,5 @@
 </geometry>
 <material name="wheel_material">
-<color rgba="0.93784246287025563316 0.77727352216680201114 0.24802940574315235356 1.0"/>
+<color rgba="0.93817637743758997004 0.77716387406765596868 0.24699191181720780985 1.0"/>
 </material>
 </visual>
@@ -70,7 +48,7 @@
 </collision>
 <inertial>
-<origin xyz="-9.458891716058550513e-06 -8.8415141495199108814e-06 -0.0151311253427085287" rpy="0 0 0"/>
-<mass value="0.019223052335254623563" />
-<inertia ixx="5.399262953463331145e-06" ixy="-7.3246329002135682946e-08"  ixz="-1.2642889979754722209e-09" iyy="5.6557979176500377362e-06" iyz="1.9098649289524929031e-09" izz="8.6846392930505483386e-06" />
+<origin xyz="-9.4080772161778185937e-06 -8.7940150929699637965e-06 -0.015171785857257018976" rpy="0 0 0"/>
+<mass value="0.019326877652137152558" />
+<inertia ixx="5.4075632337239984917e-06" ixy="-8.0312945992185011218e-08"  ixz="-1.2568956473773278438e-09" iyy="5.6885776482218881875e-06" iyz="1.916775893006806247e-09" izz="8.7138700444652767682e-06" />
 </inertial>
 </link>
@@ -92,11 +70,11 @@
 </collision>
 <inertial>
-<origin xyz="4.0756135754373242931e-11 8.4957117021027906659e-11 2.4283851137571838313e-11" rpy="0 0 0"/>
-<mass value="0.0037899803393768708749" />
-<inertia ixx="1.8303635244743846252e-07" ixy="4.2716081056736456509e-16"  ixz="-1.7514569688045876161e-15" iyy="1.8303636075213773613e-07" iyz="-3.3429142877220179384e-15" izz="9.8097062080638907831e-08" />
-</inertial>
-</link>
-<joint name="roller2_1" type="continuous">
-<origin xyz="0.020681564833504317152 -0.021119421197575767579 -0.010000000285351307028" rpy="1.570796326794896336 -0.6597090063277464278 2.3457233385922444668" />
+<origin xyz="4.0756121985606166103e-11 8.4957113535403680068e-11 2.4283847745025522076e-11" rpy="0 0 0"/>
+<mass value="0.0037899803393768713086" />
+<inertia ixx="1.8303635244743848899e-07" ixy="4.2716078955510298828e-16"  ixz="-1.7514569824195878747e-15" iyy="1.8303636075213773613e-07" iyz="-3.3429143070510763521e-15" izz="9.80970620806389343e-08" />
+</inertial>
+</link>
+<joint name="roller1_1" type="continuous">
+<origin xyz="0.020681564833508855189 -0.02111942119757877559 -0.010000000285350446605" rpy="-2.3666656417924341049 -1.5707963267948408248 0" />
 <parent link="wheel" />
 <child link="roller" />
@@ -122,11 +100,11 @@
 </collision>
 <inertial>
-<origin xyz="4.0756121876585422192e-11 8.4957096204346194938e-11 2.4283853305976183284e-11" rpy="0 0 0"/>
-<mass value="0.0037899803393768708749" />
-<inertia ixx="1.8303635244743851546e-07" ixy="4.2716078408569811146e-16"  ixz="-1.7514569733174652173e-15" iyy="1.8303636075213768319e-07" iyz="-3.3429142998677468145e-15" izz="9.80970620806389343e-08" />
-</inertial>
-</link>
-<joint name="roller2_2" type="continuous">
-<origin xyz="0.028630754033681701104 0.0073511498047736482941 -0.01000000048162325017" rpy="-1.57079632679489678 -0.95923833802399638415 -2.8902645323988411796" />
+<origin xyz="4.0756118516159214149e-11 8.4957103127062837132e-11 2.4283847745025522076e-11" rpy="0 0 0"/>
+<mass value="0.0037899803393768713086" />
+<inertia ixx="1.8303635244743848899e-07" ixy="4.2716081400933962448e-16"  ixz="-1.7514569930109819052e-15" iyy="1.8303636075213778907e-07" iyz="-3.3429142993269262604e-15" izz="9.8097062080638907831e-08" />
+</inertial>
+</link>
+<joint name="roller1_2" type="continuous">
+<origin xyz="-0.0082858436691605717728 -0.028375035936993940611 -0.010000003715208427568" rpy="1.5707963267948643615 0.039422984638921319822 -1.8430676189349126659" />
 <parent link="wheel" />
 <child link="roller_2" />
@@ -152,11 +130,11 @@
 </collision>
 <inertial>
-<origin xyz="4.0756135754373249393e-11 8.4957089265452303955e-11 2.4283849402848352643e-11" rpy="0 0 0"/>
-<mass value="0.0037899803393768708749" />
-<inertia ixx="1.8303635244743851546e-07" ixy="4.2716080577552380755e-16"  ixz="-1.7514569792812796932e-15" iyy="1.8303636075213778907e-07" iyz="-3.3429143173382564297e-15" izz="9.80970620806389343e-08" />
-</inertial>
-</link>
-<joint name="roller2_3" type="continuous">
-<origin xyz="0.020599080645981818899 0.021035055769849139717 -0.024199995144404309877" rpy="1.570796326794896558 -1.0050751734414828942 0.79586976703605405437" />
+<origin xyz="4.0756108107818351826e-11 8.4957117004850644947e-11 2.4283842540855090915e-11" rpy="0 0 0"/>
+<mass value="0.0037899803393768713086" />
+<inertia ixx="1.8303635244743848899e-07" ixy="4.2716079021680908052e-16"  ixz="-1.7514569817847873628e-15" iyy="1.8303636075213778907e-07" iyz="-3.3429143100435409156e-15" izz="9.80970620806389343e-08" />
+</inertial>
+</link>
+<joint name="roller1_3" type="continuous">
+<origin xyz="0.028630754033684657073 0.00735114980477863042 -0.010000000481622278725" rpy="-1.5707963267948972241 -0.47506888631430066461 -2.8902645323988251924" />
 <parent link="wheel" />
 <child link="roller_3" />
@@ -182,11 +160,11 @@
 </collision>
 <inertial>
-<origin xyz="4.0756135754373249393e-11 8.4957103143240124694e-11 2.4283847668124879897e-11" rpy="0 0 0"/>
-<mass value="0.0037899803393768708749" />
-<inertia ixx="1.8303635244743851546e-07" ixy="4.2716080872768029044e-16"  ixz="-1.7514569753815174093e-15" iyy="1.8303636075213789495e-07" iyz="-3.3429143089350225275e-15" izz="9.8097062080638907831e-08" />
-</inertial>
-</link>
-<joint name="roller2_4" type="continuous">
-<origin xyz="0.0079490519369571598085 0.028470515462351391606 -0.00999999706275848943" rpy="1.570796326794896558 1.0765431582887567963 -1.8430676189349801675" />
+<origin xyz="4.0756121985606166103e-11 8.4957103127062837132e-11 2.4283849479748998053e-11" rpy="0 0 0"/>
+<mass value="0.0037899803393768713086" />
+<inertia ixx="1.8303635244743848899e-07" ixy="4.2716081400933962448e-16"  ixz="-1.7514569930109819052e-15" iyy="1.8303636075213778907e-07" iyz="-3.3429142993269262604e-15" izz="9.8097062080638907831e-08" />
+</inertial>
+</link>
+<joint name="roller1_4" type="continuous">
+<origin xyz="0.0079490519369558119284 0.028470515462359964609 -0.0099999970627584200411" rpy="1.5707963267948643615 0.039422984638921319822 -1.8430676189349126659" />
 <parent link="wheel" />
 <child link="roller_4" />
@@ -212,11 +190,11 @@
 </collision>
 <inertial>
-<origin xyz="4.0756107998797633764e-11 8.4957103143240098845e-11 2.4283849402848359105e-11" rpy="0 0 0"/>
-<mass value="0.0037899803393768708749" />
-<inertia ixx="1.8303635244743851546e-07" ixy="4.2716080994071185231e-16"  ixz="-1.7514569732463042444e-15" iyy="1.8303636075213773613e-07" iyz="-3.342914303254452504e-15" izz="9.80970620806389343e-08" />
-</inertial>
-</link>
-<joint name="roller2_5" type="continuous">
-<origin xyz="-0.0079173874319013633205 0.028356888222933061133 -0.024199999101464753082" rpy="1.57079632679489678 -1.0027977690887008855 1.8430678811938736583" />
+<origin xyz="4.0756115046712262196e-11 8.4957103127062824208e-11 2.4283854683919425983e-11" rpy="0 0 0"/>
+<mass value="0.0037899803393768713086" />
+<inertia ixx="1.8303635244743848899e-07" ixy="4.2716080854478915115e-16"  ixz="-1.7514569891076034829e-15" iyy="1.8303636075213773613e-07" iyz="-3.3429142971992106269e-15" izz="9.80970620806389343e-08" />
+</inertial>
+</link>
+<joint name="roller1_5" type="continuous">
+<origin xyz="-0.0079173874319016183249 0.028356888222940322686 -0.024199999101467722928" rpy="1.5707963267948528152 -0.035629031643070047108 1.8430678811939340545" />
 <parent link="wheel" />
 <child link="roller_5" />
@@ -242,11 +220,11 @@
 </collision>
 <inertial>
-<origin xyz="4.0756114937691531209e-11 8.4957117021027906659e-11 2.4283851137571825389e-11" rpy="0 0 0"/>
-<mass value="0.0037899803393768708749" />
-<inertia ixx="1.8303635244743846252e-07" ixy="4.2716080626824243395e-16"  ixz="-1.7514569688045876161e-15" iyy="1.8303636075213773613e-07" iyz="-3.3429143197438218903e-15" izz="9.8097062080638907831e-08" />
-</inertial>
-</link>
-<joint name="roller2_6" type="continuous">
-<origin xyz="-0.020681651273558431664 0.021119338664790682225 -0.010000000622266080885" rpy="1.57079632679489678 0.6597090063277464278 -0.7958693149975488712" />
+<origin xyz="4.0756108324658792785e-11 8.4957130882638452761e-11 2.4283856418642898729e-11" rpy="0 0 0"/>
+<mass value="0.0037899803393768713086" />
+<inertia ixx="1.8303635244743843605e-07" ixy="4.2716084048573347974e-16"  ixz="-1.7514569913609862364e-15" iyy="1.8303636075213778907e-07" iyz="-3.3429143316136009109e-15" izz="9.80970620806389343e-08" />
+</inertial>
+</link>
+<joint name="roller1_6" type="continuous">
+<origin xyz="-0.020681651273562914189 0.02111933866479353411 -0.010000000622266469463" rpy="1.5707963267948510389 0.3237658697658820639 -0.79586931499757518349" />
 <parent link="wheel" />
 <child link="roller_6" />
@@ -272,11 +250,11 @@
 </collision>
 <inertial>
-<origin xyz="4.0756121876585441579e-11 8.4957103143240098845e-11 2.42838446323588034e-11" rpy="0 0 0"/>
-<mass value="0.0037899803393768708749" />
-<inertia ixx="1.8303635244743851546e-07" ixy="4.2716080414299874534e-16"  ixz="-1.7514569734306507828e-15" iyy="1.8303636075213773613e-07" iyz="-3.3429142965122737061e-15" izz="9.8097062080638907831e-08" />
-</inertial>
-</link>
-<joint name="roller2_7" type="continuous">
-<origin xyz="-0.028516458158703433812 0.0073218567028481632009 -0.024199999573447886214" rpy="-1.570796326794896558 -0.029118128194412656179 -0.25132764401667873067" />
+<origin xyz="4.0756108107818358288e-11 8.4957089249275029318e-11 2.4283846010302052562e-11" rpy="0 0 0"/>
+<mass value="0.0037899803393768713086" />
+<inertia ixx="1.8303635244743848899e-07" ixy="4.27160807953453889e-16"  ixz="-1.7514569860326745559e-15" iyy="1.8303636075213778907e-07" iyz="-3.3429143076502848406e-15" izz="9.809706208063898724e-08" />
+</inertial>
+</link>
+<joint name="roller1_7" type="continuous">
+<origin xyz="-0.028516458158707243264 0.0073218567028522536788 -0.02419999957345192465" rpy="1.5707963267947924191 0.4998755173783210326 2.8902650095730839652" />
 <parent link="wheel" />
 <child link="roller_7" />
@@ -302,11 +280,11 @@
 </collision>
 <inertial>
-<origin xyz="4.0756107998797633764e-11 8.4957096204346207862e-11 2.428385634174225655e-11" rpy="0 0 0"/>
-<mass value="0.0037899803393768708749" />
-<inertia ixx="1.8303635244743851546e-07" ixy="4.2716080577552380755e-16"  ixz="-1.7514569792812796932e-15" iyy="1.8303636075213778907e-07" iyz="-3.3429143173382564297e-15" izz="9.80970620806389343e-08" />
-</inertial>
-</link>
-<joint name="roller2_8" type="continuous">
-<origin xyz="-0.02059908211981235221 -0.021035064443088044572 -0.02419999841828643361" rpy="1.570796326794896558 -1.0050751734414828942 0.79586976703605405437" />
+<origin xyz="4.0756115046712255733e-11 8.4957103127062824208e-11 2.4283852949195953238e-11" rpy="0 0 0"/>
+<mass value="0.0037899803393768713086" />
+<inertia ixx="1.8303635244743848899e-07" ixy="4.2716078518960338886e-16"  ixz="-1.7514569807358372422e-15" iyy="1.8303636075213773613e-07" iyz="-3.3429142987394990152e-15" izz="9.80970620806389343e-08" />
+</inertial>
+</link>
+<joint name="roller1_8" type="continuous">
+<origin xyz="-0.02851643393617246669 -0.0073217973661822786241 -0.010000001453654761008" rpy="-1.5707963267947111508 -0.47506888631359656117 -2.8902645323989122339" />
 <parent link="wheel" />
 <child link="roller_8" />
@@ -332,11 +310,11 @@
 </collision>
 <inertial>
-<origin xyz="4.0756135754373230006e-11 8.4957117021027906659e-11 2.4283848535486617886e-11" rpy="0 0 0"/>
-<mass value="0.0037899803393768708749" />
-<inertia ixx="1.8303635244743851546e-07" ixy="4.2716076857917792248e-16"  ixz="-1.751456967687839831e-15" iyy="1.8303636075213773613e-07" iyz="-3.3429143078393905768e-15" izz="9.80970620806389343e-08" />
-</inertial>
-</link>
-<joint name="roller2_9" type="continuous">
-<origin xyz="-0.028516433936169462149 -0.0073217973661773502747 -0.010000001453652984651" rpy="-1.570796326794896558 -0.95923833802399638415 -2.8902645323988411796" />
+<origin xyz="4.0756108107818358288e-11 8.4957103127062837132e-11 2.4283852949195953238e-11" rpy="0 0 0"/>
+<mass value="0.0037899803393768713086" />
+<inertia ixx="1.8303635244743848899e-07" ixy="4.2716081252639028129e-16"  ixz="-1.7514569804702362556e-15" iyy="1.8303636075213778907e-07" iyz="-3.3429142988320809143e-15" izz="9.80970620806389343e-08" />
+</inertial>
+</link>
+<joint name="roller1_9" type="continuous">
+<origin xyz="-0.020599082119815405323 -0.021035064443091409936 -0.024199998418290208368" rpy="1.5707963267949525132 -0.33636312788316474753 0.79586976703607825723" />
 <parent link="wheel" />
 <child link="roller_9" />
@@ -362,11 +340,11 @@
 </collision>
 <inertial>
-<origin xyz="4.0756149632161057208e-11 8.4957096204346220787e-11 2.4283849402848355874e-11" rpy="0 0 0"/>
-<mass value="0.0037899803393768708749" />
-<inertia ixx="1.8303635244743851546e-07" ixy="4.2716080872768029044e-16"  ixz="-1.7514569753815174093e-15" iyy="1.8303636075213789495e-07" iyz="-3.3429143089350225275e-15" izz="9.8097062080638907831e-08" />
-</inertial>
-</link>
-<joint name="roller2_10" type="continuous">
-<origin xyz="-0.0082858436691589446021 -0.028375035936988014795 -0.010000003715208150012" rpy="1.570796326794896558 1.0765431582887567963 -1.8430676189349801675" />
+<origin xyz="4.0756118516159207687e-11 8.4957075371487221503e-11 2.4283849479749001284e-11" rpy="0 0 0"/>
+<mass value="0.0037899803393768713086" />
+<inertia ixx="1.8303635244743843605e-07" ixy="4.2716080311549494243e-16"  ixz="-1.7514569794927228148e-15" iyy="1.8303636075213778907e-07" iyz="-3.3429142912277513e-15" izz="9.80970620806389343e-08" />
+</inertial>
+</link>
+<joint name="roller1_10" type="continuous">
+<origin xyz="0.0079173979793267165728 -0.028356884977344593013 -0.024199999508979525009" rpy="1.5707963267949405228 0.03562903164307248266 -1.2985247723958603938" />
 <parent link="wheel" />
 <child link="roller_10" />
@@ -392,11 +370,11 @@
 </collision>
 <inertial>
-<origin xyz="4.0756135754373249393e-11 8.4957110082134002752e-11 2.4283852872295304596e-11" rpy="0 0 0"/>
-<mass value="0.0037899803393768708749" />
-<inertia ixx="1.8303635244743851546e-07" ixy="4.2716080511422067532e-16"  ixz="-1.7514569745051181871e-15" iyy="1.8303636075213773613e-07" iyz="-3.342914314594920451e-15" izz="9.80970620806389343e-08" />
-</inertial>
-</link>
-<joint name="roller2_11" type="continuous">
-<origin xyz="0.0079173979793228238533 -0.028356884977337862286 -0.024199999508976485774" rpy="1.570796326794896558 1.0027977690887006634 -1.2985247723959187915" />
+<origin xyz="4.0756121985606172565e-11 8.4957103127062837132e-11 2.4283852949195946775e-11" rpy="0 0 0"/>
+<mass value="0.0037899803393768713086" />
+<inertia ixx="1.8303635244743859487e-07" ixy="4.2716080665760632879e-16"  ixz="-1.7514569880785997103e-15" iyy="1.8303636075213778907e-07" iyz="-3.3429143104060729886e-15" izz="9.80970620806389343e-08" />
+</inertial>
+</link>
+<joint name="roller1_11" type="continuous">
+<origin xyz="0.028516471920458755923 -0.0073217858682538168591 -0.024199999328584992364" rpy="1.5707963267949687225 0.49987551737898944237 2.8902650095731661217" />
 <parent link="wheel" />
 <child link="roller_11" />
@@ -422,11 +400,11 @@
 </collision>
 <inertial>
-<origin xyz="4.0756128815479345486e-11 8.495710314324011177e-11 2.4283853739657042585e-11" rpy="0 0 0"/>
-<mass value="0.0037899803393768708749" />
-<inertia ixx="1.8303635244743851546e-07" ixy="4.2716081765933730457e-16"  ixz="-1.7514569739582738912e-15" iyy="1.8303636075213778907e-07" iyz="-3.3429143227896726155e-15" izz="9.80970620806389343e-08" />
-</inertial>
-</link>
-<joint name="roller2_12" type="continuous">
-<origin xyz="0.028516471920454564831 -0.0073217858682495711234 -0.024199999328582064151" rpy="-1.570796326794896558 -0.029118128194412718629 -0.25132764401667873067" />
+<origin xyz="4.0756115914074019571e-11 8.4957130882638439836e-11 2.428385121447247403e-11" rpy="0 0 0"/>
+<mass value="0.0037899803393768713086" />
+<inertia ixx="1.8303635244743859487e-07" ixy="4.2716081974557339914e-16"  ixz="-1.7514569668193931157e-15" iyy="1.8303636075213773613e-07" iyz="-3.3429143129522359451e-15" izz="9.80970620806389343e-08" />
+</inertial>
+</link>
+<joint name="roller1_" type="continuous">
+<origin xyz="0.020599080645985489574 0.021035055769852671614 -0.024199995144406849512" rpy="1.5707963267948636954 -0.33636312788368860627 0.7958697670360835863" />
 <parent link="wheel" />
 <child link="roller_12" />
@@ -435,6 +413,6 @@
 <joint_properties friction="0.0"/>
 </joint>
-<joint name="wheel2" type="continuous">
-<origin xyz="1.6916223843148240913e-18 0.015229328657860304735 2.999999999994673594e-05" rpy="3.141592653589793116 -3.460379863012290867e-16 1.570796326794896558" />
+<joint name="wheel1" type="continuous">
+<origin xyz="-0.10382679491924297344 -0.059944427995721236146 0.017831400000000004191" rpy="1.570796326794896558 1.1830378826286079221e-16 2.0943951023931974831" />
 <parent link="motor" />
 <child link="wheel" />
@@ -443,851 +421,3 @@
 <joint_properties friction="0.0"/>
 </joint>
-<joint name="motor1" type="fixed">
-<origin xyz="0.073581777378123131017 -0.041158680771919600727 2.6020852139652106416e-17" rpy="-1.570796326794896336 -1.660721004497953203e-16 -2.0807970750313837804" />
-<parent link="base" />
-<child link="motor" />
-<axis xyz="0 0 1"/>
-<limit effort="1" velocity="20" />
-<joint_properties friction="0.0"/>
-</joint>
-<link name="motor_2">
-<visual>
-<origin xyz="0 0 0" rpy="0 -0 0" />
-<geometry>
-<mesh filename="package://omnibot_description/meshes/motor.stl"/>
-</geometry>
-<material name="motor_2_material">
-<color rgba="0.90196078431372550543 0.91764705882352937127 0.92941176470588238168 1.0"/>
-</material>
-</visual>
-<collision>
-<origin xyz="0 0 0" rpy="0 -0 0" />
-<geometry>
-<mesh filename="package://omnibot_description/meshes/motor.stl"/>
-</geometry>
-</collision>
-<inertial>
-<origin xyz="-2.0988305528216905668e-06 0.015050377580170260991 -0.021659280060218957797" rpy="0 0 0"/>
-<mass value="0.12860494827495119741" />
-<inertia ixx="4.6506247208995520883e-05" ixy="1.6921131916578120212e-09"  ixz="-3.4608427741392125582e-09" iyy="4.6246527094885930766e-05" iyz="1.0074294037198133834e-06" izz="1.066124497744399909e-05" />
-</inertial>
-</link>
-<link name="wheel_2">
-<visual>
-<origin xyz="0 0 0" rpy="0 -0 0" />
-<geometry>
-<mesh filename="package://omnibot_description/meshes/wheel.stl"/>
-</geometry>
-<material name="wheel_2_material">
-<color rgba="0.93784246287025563316 0.77727352216680201114 0.24802940574315235356 1.0"/>
-</material>
-</visual>
-<collision>
-<origin xyz="0 0 0" rpy="0 -0 0" />
-<geometry>
-<mesh filename="package://omnibot_description/meshes/wheel.stl"/>
-</geometry>
-</collision>
-<inertial>
-<origin xyz="-9.4588917159859343785e-06 -8.841514149794161515e-06 -0.015131125342709179221" rpy="0 0 0"/>
-<mass value="0.019223052335254623563" />
-<inertia ixx="5.3992629534639359265e-06" ixy="-7.3246329002134650625e-08"  ixz="-1.2642889980048470588e-09" iyy="5.655797917650546803e-06" iyz="1.9098649291002472128e-09" izz="8.6846392930512276591e-06" />
-</inertial>
-</link>
-<link name="roller_13">
-<visual>
-<origin xyz="0 0 0" rpy="0 -0 0" />
-<geometry>
-<mesh filename="package://omnibot_description/meshes/roller.stl"/>
-</geometry>
-<material name="roller_13_material">
-<color rgba="0.098039215686274508443 0.098039215686274508443 0.098039215686274508443 1.0"/>
-</material>
-</visual>
-<collision>
-<origin xyz="0 0 0" rpy="0 -0 0" />
-<geometry>
-<mesh filename="package://omnibot_description/meshes/roller.stl"/>
-</geometry>
-</collision>
-<inertial>
-<origin xyz="4.0756121876585435117e-11 8.4957103143240098845e-11 2.4283851137571844776e-11" rpy="0 0 0"/>
-<mass value="0.0037899803393768708749" />
-<inertia ixx="1.8303635244743846252e-07" ixy="4.2716080820167912941e-16"  ixz="-1.7514569759688257337e-15" iyy="1.8303636075213773613e-07" iyz="-3.3429143027409348202e-15" izz="9.809706208063898724e-08" />
-</inertial>
-</link>
-<joint name="roller1_1" type="continuous">
-<origin xyz="0.020681564833506995565 -0.021119421197577783328 -0.010000000285350016394" rpy="-0.7749270117973218186 1.5707963267948548136 0" />
-<parent link="wheel_2" />
-<child link="roller_13" />
-<axis xyz="0 0 1"/>
-<limit effort="1" velocity="20" />
-<joint_properties friction="0.0"/>
-</joint>
-<link name="roller_14">
-<visual>
-<origin xyz="0 0 0" rpy="0 -0 0" />
-<geometry>
-<mesh filename="package://omnibot_description/meshes/roller.stl"/>
-</geometry>
-<material name="roller_14_material">
-<color rgba="0.098039215686274508443 0.098039215686274508443 0.098039215686274508443 1.0"/>
-</material>
-</visual>
-<collision>
-<origin xyz="0 0 0" rpy="0 -0 0" />
-<geometry>
-<mesh filename="package://omnibot_description/meshes/roller.stl"/>
-</geometry>
-</collision>
-<inertial>
-<origin xyz="4.0756121876585441579e-11 8.495708926545229103e-11 2.4283847668124883128e-11" rpy="0 0 0"/>
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