Commit message: Wheels roling, rollers not yet usable

File: src/omnibot_description/urdf/omnibot_gazebo.xacro (robot description, xacro)
@@ -13,4 +13,15 @@
     <xacro:transmission id="2"/>
     <xacro:transmission id="3"/>
+    <xacro:macro name="roller_link_values" params="wheel_id id">
+        <gazebo reference="roller_${wheel_id}_${id}_link">
+            <mu1>100000000000000.0</mu1>
+            <mu2>100000000000000.0</mu2>
+            <kp>10000000000000.0</kp>
+            <kd>10.0</kd>
+            <minDepth>0.001</minDepth>
+            <maxVel>0.1</maxVel>
+            <fdir1>1 0 0</fdir1>
+        </gazebo>
+    </xacro:macro>
     <xacro:macro name="wheel_link_values" params="id">
         <gazebo reference="wheel_${id}_link">
@@ -23,4 +34,16 @@
             <fdir1>1 0 0</fdir1>
         </gazebo>
+        <xacro:roller_link_values id="1" wheel_id="${id}"/>
+        <xacro:roller_link_values id="2" wheel_id="${id}"/>
+        <xacro:roller_link_values id="3" wheel_id="${id}"/>
+        <xacro:roller_link_values id="4" wheel_id="${id}"/>
+        <xacro:roller_link_values id="5" wheel_id="${id}"/>
+        <xacro:roller_link_values id="6" wheel_id="${id}"/>
+        <xacro:roller_link_values id="7" wheel_id="${id}"/>
+        <xacro:roller_link_values id="8" wheel_id="${id}"/>
+        <xacro:roller_link_values id="9" wheel_id="${id}"/>
+        <xacro:roller_link_values id="10" wheel_id="${id}"/>
+        <xacro:roller_link_values id="11" wheel_id="${id}"/>
+        <xacro:roller_link_values id="12" wheel_id="${id}"/>
     </xacro:macro>
     <xacro:wheel_link_values id="1"/>

File: src/omnibot_description/urdf/roller.xacro (robot description, xacro)
@@ -4,6 +4,6 @@
         <color rgba="0 1 0 1.0"/>
     </material>
-    <xacro:macro name="roller" params="id parent_id pitch x y z">
-        <link name="roller_${parent_id}_${id}_link">
+    <xacro:macro name="roller" params="id wheel_id pitch x y z">
+        <link name="roller_${wheel_id}_${id}_link">
             <inertial>
                 <mass value="1.0"/>
@@ -23,9 +23,8 @@
                     <mesh filename="package://omnibot_description/meshes/wheel/colision_omni_roller.stl"/>
                 </geometry>
-            </collision>
         </link>
-        <joint name="roller_${parent_id}_${id}_joint" type="continuous">
-            <parent link="wheel_${parent_id}_link"/>
-            <child link="roller_${parent_id}_${id}_link"/>
+        <joint name="roller_${wheel_id}_${id}_joint" type="continuous">
+            <parent link="wheel_${wheel_id}_link"/>
+            <child link="roller_${wheel_id}_${id}_link"/>
             <axis xyz="0 0 1"/>
             <origin rpy="0 ${pitch} 0" xyz="${x} ${y} ${z}"/>

File: src/omnibot_description/urdf/wheel.xacro (robot description, xacro)
@@ -27,16 +27,16 @@
             <origin rpy="0 0 ${yaw}" xyz="${x} ${y} -0.0124"/>
         </joint>
-        <xacro:roller id="1" parent_id="${id}" pitch="-0.257" x="-0.0285" y="-0.002" z="-0.0075"/>
-        <xacro:roller id="2" parent_id="${id}" pitch="-1.3" x="-0.0079" y="-0.002" z="-0.0283"/>
-        <xacro:roller id="3" parent_id="${id}" pitch="0.789" x="0.0206" y="-0.002" z="-0.0208"/>
-        <xacro:roller id="4" parent_id="${id}" pitch="-0.257" x="0.0285" y="-0.002" z="0.0075"/>
-        <xacro:roller id="5" parent_id="${id}" pitch="-1.3" x="0.0079" y="-0.002" z="0.0283"/>
-        <xacro:roller id="6" parent_id="${id}" pitch="0.789" x="-0.0206" y="-0.002" z="0.0208"/>
-        <xacro:roller id="7" parent_id="${id}" pitch="0.25" x="-0.0286" y="0.0122" z="0.0075"/>
-        <xacro:roller id="8" parent_id="${id}" pitch="-0.8" x="-0.0205" y="0.0122" z="-0.021"/>
-        <xacro:roller id="9" parent_id="${id}" pitch="-1.85" x="0.008" y="0.0122" z="-0.0285"/>
-        <xacro:roller id="10" parent_id="${id}" pitch="0.25" x="0.0286" y="0.0122" z="-0.0075"/>
-        <xacro:roller id="11" parent_id="${id}" pitch="-0.8" x="0.0205" y="0.0122" z="0.021"/>
-        <xacro:roller id="12" parent_id="${id}" pitch="-1.85" x="-0.008" y="0.0122" z="0.0285"/>
+        <xacro:roller wheel_id="${id}" id="1" pitch="-0.257" x="-0.0285" y="-0.002" z="-0.0075"/>
+        <xacro:roller wheel_id="${id}" id="2" pitch="-1.3" x="-0.0079" y="-0.002" z="-0.0283"/>
+        <xacro:roller wheel_id="${id}" id="3" pitch="0.789" x="0.0206" y="-0.002" z="-0.0208"/>
+        <xacro:roller wheel_id="${id}" id="4" pitch="-0.257" x="0.0285" y="-0.002" z="0.0075"/>
+        <xacro:roller wheel_id="${id}" id="5" pitch="-1.3" x="0.0079" y="-0.002" z="0.0283"/>
+        <xacro:roller wheel_id="${id}" id="6" pitch="0.789" x="-0.0206" y="-0.002" z="0.0208"/>
+        <xacro:roller wheel_id="${id}" id="7" pitch="0.25" x="-0.0286" y="0.0122" z="0.0075"/>
+        <xacro:roller wheel_id="${id}" id="8" pitch="-0.8" x="-0.0205" y="0.0122" z="-0.021"/>
+        <xacro:roller wheel_id="${id}" id="9" pitch="-1.85" x="0.008" y="0.0122" z="-0.0285"/>
+        <xacro:roller wheel_id="${id}" id="10" pitch="0.25" x="0.0286" y="0.0122" z="-0.0075"/>
+        <xacro:roller wheel_id="${id}" id="11" pitch="-0.8" x="0.0205" y="0.0122" z="0.021"/>
+        <xacro:roller wheel_id="${id}" id="12" pitch="-1.85" x="-0.008" y="0.0122" z="0.0285"/>
     </xacro:macro>
 </robot>

Commit message: plugins up and runing

File: src/omnibot_description/urdf/omnibot_gazebo.xacro (robot description, xacro)
@@ -13,6 +13,6 @@
     <xacro:transmission id="2"/>
     <xacro:transmission id="3"/>
-    <xacro:macro name="roller_link_values" params="wheel_id id">
-        <gazebo reference="roller_${wheel_id}_${id}_link">
+    <xacro:macro name="roller_link_values">
+        <gazebo reference="roller_${id}">
             <mu1>100000000000000.0</mu1>
             <mu2>100000000000000.0</mu2>
@@ -25,5 +25,5 @@
     </xacro:macro>
     <xacro:macro name="wheel_link_values" params="id">
-        <gazebo reference="wheel_${id}_link">
+        <gazebo reference="wheel${id}">
             <mu1>100000000000000.0</mu1>
             <mu2>100000000000000.0</mu2>
@@ -34,20 +34,55 @@
             <fdir1>1 0 0</fdir1>
         </gazebo>
-        <xacro:roller_link_values id="1" wheel_id="${id}"/>
-        <xacro:roller_link_values id="2" wheel_id="${id}"/>
-        <xacro:roller_link_values id="3" wheel_id="${id}"/>
-        <xacro:roller_link_values id="4" wheel_id="${id}"/>
-        <xacro:roller_link_values id="5" wheel_id="${id}"/>
-        <xacro:roller_link_values id="6" wheel_id="${id}"/>
-        <xacro:roller_link_values id="7" wheel_id="${id}"/>
-        <xacro:roller_link_values id="8" wheel_id="${id}"/>
-        <xacro:roller_link_values id="9" wheel_id="${id}"/>
-        <xacro:roller_link_values id="10" wheel_id="${id}"/>
-        <xacro:roller_link_values id="11" wheel_id="${id}"/>
-        <xacro:roller_link_values id="12" wheel_id="${id}"/>
     </xacro:macro>
-    <xacro:wheel_link_values id="1"/>
-    <xacro:wheel_link_values id="2"/>
-    <xacro:wheel_link_values id="3"/>
+    <xacro:wheel_link_values id=""/>
+    <xacro:wheel_link_values id="_2"/>
+    <xacro:wheel_link_values id="_3"/>
+    <xacro:macro name="roller_link_values" params="id">
+        <gazebo reference="roller${id}">
+            <mu1>100000000000000.0</mu1>
+            <mu2>100000000000000.0</mu2>
+            <kp>10000000000000.0</kp>
+            <kd>10.0</kd>
+            <minDepth>0.001</minDepth>
+            <maxVel>0.1</maxVel>
+            <fdir1>1 0 0</fdir1>
+        </gazebo>
+    </xacro:macro>
+    <xacro:roller_link_values id=""/>
+    <xacro:roller_link_values id="_2"/>
+    <xacro:roller_link_values id="_3"/>
+    <xacro:roller_link_values id="_4"/>
+    <xacro:roller_link_values id="_5"/>
+    <xacro:roller_link_values id="_6"/>
+    <xacro:roller_link_values id="_7"/>
+    <xacro:roller_link_values id="_8"/>
+    <xacro:roller_link_values id="_9"/>
+    <xacro:roller_link_values id="_10"/>
+    <xacro:roller_link_values id="_11"/>
+    <xacro:roller_link_values id="_12"/>
+    <xacro:roller_link_values id="_13"/>
+    <xacro:roller_link_values id="_14"/>
+    <xacro:roller_link_values id="_15"/>
+    <xacro:roller_link_values id="_16"/>
+    <xacro:roller_link_values id="_17"/>
+    <xacro:roller_link_values id="_18"/>
+    <xacro:roller_link_values id="_19"/>
+    <xacro:roller_link_values id="_20"/>
+    <xacro:roller_link_values id="_21"/>
+    <xacro:roller_link_values id="_22"/>
+    <xacro:roller_link_values id="_23"/>
+    <xacro:roller_link_values id="_24"/>
+    <xacro:roller_link_values id="_25"/>
+    <xacro:roller_link_values id="_26"/>
+    <xacro:roller_link_values id="_27"/>
+    <xacro:roller_link_values id="_28"/>
+    <xacro:roller_link_values id="_29"/>
+    <xacro:roller_link_values id="_30"/>
+    <xacro:roller_link_values id="_31"/>
+    <xacro:roller_link_values id="_32"/>
+    <xacro:roller_link_values id="_33"/>
+    <xacro:roller_link_values id="_34"/>
+    <xacro:roller_link_values id="_35"/>
+    <xacro:roller_link_values id="_36"/>
     <gazebo>
         <plugin filename="libgazebo_ros2_control.so" name="gazebo_ros2_control">

File: src/omnibot_description/urdf/omnibot_ros2_control.xacro (robot description, xacro)
@@ -6,5 +6,5 @@
         </hardware>
         <xacro:macro name="ros2_control" params="id">
-            <joint name="wheel_${id}_joint">
+            <joint name="wheel${id}">
                 <command_interface name="velocity">
                     <parameter name="min">-1</parameter>

Commit message: Gazebo model missing wheels

File: src/omnibot_description/urdf/omnibot_gazebo.xacro (robot description, xacro)
@@ -5,5 +5,5 @@
             <plugin>transmission_interface/SimpleTransmission</plugin>
             <actuator name="wheel_${id}_motor" role="actuator_${id}"/>
-            <joint name="wheel_${id}_joint" role="joint_${id}">
+            <joint name="wheel${id}" role="joint_${id}">
                 <mechanical_reduction>1.0</mechanical_reduction>
             </joint>
@@ -35,7 +35,7 @@
         </gazebo>
     </xacro:macro>
-    <xacro:wheel_link_values id=""/>
-    <xacro:wheel_link_values id="_2"/>
-    <xacro:wheel_link_values id="_3"/>
+    <xacro:wheel_link_values id="1"/>
+    <xacro:wheel_link_values id="1_2"/>
+    <xacro:wheel_link_values id="1_3"/>
     <xacro:macro name="roller_link_values" params="id">
         <gazebo reference="roller${id}">
@@ -49,5 +49,5 @@
         </gazebo>
     </xacro:macro>
-    <xacro:roller_link_values id=""/>
+    <xacro:roller_link_values id="_1"/>
     <xacro:roller_link_values id="_2"/>
     <xacro:roller_link_values id="_3"/>
